File: MotorController/TEMPERATURE.kicad_sch (KiCad schematic)
At the start: 0 parts

Commit message: Schematic Updates
Parts:
- added C?: 680pF, symbol Device:C_Small
- added C?: 0.1uF, symbol Device:C_Small
- added R?: 100, symbol Device:R_Small_US
- added U?: TMP236AQDBZRQ1, symbol ProjectSymbols:TMP236AQDBZRQ1
Connections:
- new net: C?.2, R?.2, U?.1 (VDD)
- new net +3V3: R?.1
- new net GND: C?.1, C?.1, U?.3 (GND)
- new net TEMP_VSENSE: C?.2, U?.2 (VOUT)
Changed lines of the file:
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@@
 (kicad_sch (version 20211123) (generator eeschema)
   (paper "A4")
+  (junction (at 123.19 92.71) (diameter 0) (color 0 0 0 0)
+  )
+  (junction (at 172.72 92.71) (diameter 0) (color 0 0 0 0)
+  )
+  (wire (pts (xy 172.72 92.71) (xy 187.96 92.71))
+    (stroke (width 0) (type default) (color 0 0 0 0))
+  )
+  (wire (pts (xy 123.19 92.71) (xy 119.38 92.71))
+    (stroke (width 0) (type default) (color 0 0 0 0))
+  )
+  (wire (pts (xy 172.72 95.25) (xy 172.72 92.71))
+    (stroke (width 0) (type default) (color 0 0 0 0))
+  )
+  (wire (pts (xy 163.83 102.87) (xy 163.83 97.79))
+    (stroke (width 0) (type default) (color 0 0 0 0))
+  )
+  (wire (pts (xy 110.49 92.71) (xy 114.3 92.71))
+    (stroke (width 0) (type default) (color 0 0 0 0))
+  )
+  (wire (pts (xy 123.19 95.25) (xy 123.19 92.71))
+    (stroke (width 0) (type default) (color 0 0 0 0))
+  )
+  (wire (pts (xy 123.19 92.71) (xy 140.97 92.71))
+    (stroke (width 0) (type default) (color 0 0 0 0))
+  )
+  (wire (pts (xy 172.72 100.33) (xy 172.72 102.87))
+    (stroke (width 0) (type default) (color 0 0 0 0))
+  )
+  (wire (pts (xy 123.19 100.33) (xy 123.19 102.87))
+    (stroke (width 0) (type default) (color 0 0 0 0))
+  )
+  (wire (pts (xy 163.83 97.79) (xy 160.02 97.79))
+    (stroke (width 0) (type default) (color 0 0 0 0))
+  )
+  (wire (pts (xy 172.72 92.71) (xy 160.02 92.71))
+    (stroke (width 0) (type default) (color 0 0 0 0))
+  )
+  (hierarchical_label "+3V3" (shape input) (at 110.49 92.71 180)
+    (effects (font (size 1.27 1.27)) (justify right))
+  )
+  (hierarchical_label "TEMP_VSENSE" (shape output) (at 187.96 92.71 0)
+    (effects (font (size 1.27 1.27)) (justify left))
+  )
+  (symbol (lib_id "ProjectSymbols:TMP236AQDBZRQ1") (at 149.86 96.52 0) (unit 1)
+    (in_bom yes) (on_board yes) (fields_autoplaced)
+    (property "Reference" "U?" (id 0) (at 150.495 86.36 0))
+    (property "Value" "TMP236AQDBZRQ1" (id 1) (at 150.495 88.9 0))
+    (property "Footprint" "" (id 2) (at 152.4 80.01 0)
+      (effects (font (size 1.27 1.27)) hide)
+    )
+    (property "Datasheet" "" (id 3) (at 152.4 80.01 0)
+      (effects (font (size 1.27 1.27)) hide)
+    )
+    (pin "1")
+    (pin "2")
+    (pin "3")
+  )
+  (symbol (lib_id "Device:R_Small_US") (at 116.84 92.71 90) (unit 1)
+    (in_bom yes) (on_board yes) (fields_autoplaced)
+    (property "Reference" "R?" (id 0) (at 116.84 86.36 90))
+    (property "Value" "100" (id 1) (at 116.84 88.9 90))
+    (property "Footprint" "" (id 2) (at 116.84 92.71 0)
+      (effects (font (size 1.27 1.27)) hide)
+    )
+    (property "Datasheet" "~" (id 3) (at 116.84 92.71 0)
+      (effects (font (size 1.27 1.27)) hide)
+    )
+    (pin "1")
+    (pin "2")
+  )
+  (symbol (lib_id "power:GND") (at 172.72 102.87 0) (unit 1)
+    (in_bom yes) (on_board yes) (fields_autoplaced)
+    (property "Reference" "#PWR?" (id 0) (at 172.72 109.22 0)
+      (effects (font (size 1.27 1.27)) hide)
+    )
+    (property "Value" "GND" (id 1) (at 172.72 107.95 0)
+      (effects (font (size 1.27 1.27)) hide)
+    )
+    (property "Footprint" "" (id 2) (at 172.72 102.87 0)
+      (effects (font (size 1.27 1.27)) hide)
+    )
+    (property "Datasheet" "" (id 3) (at 172.72 102.87 0)
+      (effects (font (size 1.27 1.27)) hide)
+    )
+    (pin "1")
+  )
+  (symbol (lib_id "Device:C_Small") (at 172.72 97.79 180) (unit 1)
+    (in_bom yes) (on_board yes) (fields_autoplaced)
+    (property "Reference" "C?" (id 0) (at 175.26 96.5135 0)
+      (effects (font (size 1.27 1.27)) (justify right))
+    )
+    (property "Value" "680pF" (id 1) (at 175.26 99.0535 0)
+      (effects (font (size 1.27 1.27)) (justify right))
+    )
+    (property "Footprint" "" (id 2) (at 172.72 97.79 0)
+      (effects (font (size 1.27 1.27)) hide)
+    )
+    (property "Datasheet" "~" (id 3) (at 172.72 97.79 0)
+      (effects (font (size 1.27 1.27)) hide)
+    )
+    (pin "1")
+    (pin "2")
+  )
+  (symbol (lib_id "Device:C_Small") (at 123.19 97.79 180) (unit 1)
+    (in_bom yes) (on_board yes) (fields_autoplaced)
+    (property "Reference" "C?" (id 0) (at 125.73 96.5135 0)
+      (effects (font (size 1.27 1.27)) (justify right))
+    )
+    (property "Value" "0.1uF" (id 1) (at 125.73 99.0535 0)
+      (effects (font (size 1.27 1.27)) (justify right))
+    )
+    (property "Footprint" "" (id 2) (at 123.19 97.79 0)
+      (effects (font (size 1.27 1.27)) hide)
+    )
+    (property "Datasheet" "~" (id 3) (at 123.19 97.79 0)
+      (effects (font (size 1.27 1.27)) hide)
+    )
+    (pin "1")
+    (pin "2")
+  )
+  (symbol (lib_id "power:GND") (at 163.83 102.87 0) (unit 1)
+    (in_bom yes) (on_board yes) (fields_autoplaced)
+    (property "Reference" "#PWR?" (id 0) (at 163.83 109.22 0)
+      (effects (font (size 1.27 1.27)) hide)
+    )
+    (property "Value" "GND" (id 1) (at 163.83 107.95 0)
+      (effects (font (size 1.27 1.27)) hide)
+    )
+    (property "Footprint" "" (id 2) (at 163.83 102.87 0)
+      (effects (font (size 1.27 1.27)) hide)
+    )
+    (property "Datasheet" "" (id 3) (at 163.83 102.87 0)
+      (effects (font (size 1.27 1.27)) hide)
+    )
+    (pin "1")
+  )
+  (symbol (lib_id "power:GND") (at 123.19 102.87 0) (unit 1)
+    (in_bom yes) (on_board yes) (fields_autoplaced)
+    (property "Reference" "#PWR?" (id 0) (at 123.19 109.22 0)
+      (effects (font (size 1.27 1.27)) hide)
+    )
+    (property "Value" "GND" (id 1) (at 123.19 107.95 0)
+      (effects (font (size 1.27 1.27)) hide)
+    )
+    (property "Footprint" "" (id 2) (at 123.19 102.87 0)
+      (effects (font (size 1.27 1.27)) hide)
+    )
+    (property "Datasheet" "" (id 3) (at 123.19 102.87 0)
+      (effects (font (size 1.27 1.27)) hide)
+    )
+    (pin "1")
+  )
 )

Commit message: Updates
Parts:
- C12: renamed from C?; footprint (none) -> Capacitor_SMD:C_0603_1608Metric; MPN (none) -> CC0603JRX7R8BB104
- C13: renamed from C?; footprint (none) -> Capacitor_SMD:C_0603_1608Metric; MPN (none) -> CC0603JRNPO8BN681
- R13: renamed from R?; footprint (none) -> Resistor_SMD:R_0603_1608Metric; MPN (none) -> RC0603FR-07100RL
- U7: renamed from U?; footprint (none) -> Package_TO_SOT_SMD:SC-59; MPN (none) -> TMP236AQDBZRQ1
Changed lines of the file:
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@@
   (symbol (lib_id "ProjectSymbols:TMP236AQDBZRQ1") (at 149.86 96.52 0) (unit 1)
     (in_bom yes) (on_board yes) (fields_autoplaced)
-    (property "Reference" "U?" (id 0) (at 150.495 86.36 0))
+    (property "Reference" "U7" (id 0) (at 150.495 86.36 0))
     (property "Value" "TMP236AQDBZRQ1" (id 1) (at 150.495 88.9 0))
-    (property "Footprint" "" (id 2) (at 152.4 80.01 0)
+    (property "Footprint" "Package_TO_SOT_SMD:SC-59" (id 2) (at 152.4 80.01 0)
       (effects (font (size 1.27 1.27)) hide)
     )
     (property "Datasheet" "" (id 3) (at 152.4 80.01 0)
+      (effects (font (size 1.27 1.27)) hide)
+    )
+    (property "MPN" "TMP236AQDBZRQ1" (id 4) (at 149.86 96.52 0)
       (effects (font (size 1.27 1.27)) hide)
     )
@@
   (symbol (lib_id "Device:R_Small_US") (at 116.84 92.71 90) (unit 1)
     (in_bom yes) (on_board yes) (fields_autoplaced)
-    (property "Reference" "R?" (id 0) (at 116.84 86.36 90))
+    (property "Reference" "R13" (id 0) (at 116.84 86.36 90))
     (property "Value" "100" (id 1) (at 116.84 88.9 90))
-    (property "Footprint" "" (id 2) (at 116.84 92.71 0)
+    (property "Footprint" "Resistor_SMD:R_0603_1608Metric" (id 2) (at 116.84 92.71 0)
       (effects (font (size 1.27 1.27)) hide)
     )
     (property "Datasheet" "~" (id 3) (at 116.84 92.71 0)
+      (effects (font (size 1.27 1.27)) hide)
+    )
+    (property "MPN" "RC0603FR-07100RL" (id 4) (at 116.84 92.71 0)
       (effects (font (size 1.27 1.27)) hide)
     )
@@
   (symbol (lib_id "power:GND") (at 172.72 102.87 0) (unit 1)
     (in_bom yes) (on_board yes) (fields_autoplaced)
-    (property "Reference" "#PWR?" (id 0) (at 172.72 109.22 0)
+    (property "Reference" "#PWR025" (id 0) (at 172.72 109.22 0)
       (effects (font (size 1.27 1.27)) hide)
     )
@@
   (symbol (lib_id "Device:C_Small") (at 172.72 97.79 180) (unit 1)
     (in_bom yes) (on_board yes) (fields_autoplaced)
-    (property "Reference" "C?" (id 0) (at 175.26 96.5135 0)
+    (property "Reference" "C13" (id 0) (at 175.26 96.5135 0)
       (effects (font (size 1.27 1.27)) (justify right))
     )
@@
       (effects (font (size 1.27 1.27)) (justify right))
     )
-    (property "Footprint" "" (id 2) (at 172.72 97.79 0)
+    (property "Footprint" "Capacitor_SMD:C_0603_1608Metric" (id 2) (at 172.72 97.79 0)
       (effects (font (size 1.27 1.27)) hide)
     )
     (property "Datasheet" "~" (id 3) (at 172.72 97.79 0)
+      (effects (font (size 1.27 1.27)) hide)
+    )
+    (property "MPN" "CC0603JRNPO8BN681" (id 4) (at 172.72 97.79 0)
       (effects (font (size 1.27 1.27)) hide)
     )
@@
   (symbol (lib_id "Device:C_Small") (at 123.19 97.79 180) (unit 1)
     (in_bom yes) (on_board yes) (fields_autoplaced)
-    (property "Reference" "C?" (id 0) (at 125.73 96.5135 0)
+    (property "Reference" "C12" (id 0) (at 125.73 96.5135 0)
       (effects (font (size 1.27 1.27)) (justify right))
     )
@@
       (effects (font (size 1.27 1.27)) (justify right))
     )
-    (property "Footprint" "" (id 2) (at 123.19 97.79 0)
+    (property "Footprint" "Capacitor_SMD:C_0603_1608Metric" (id 2) (at 123.19 97.79 0)
       (effects (font (size 1.27 1.27)) hide)
     )
     (property "Datasheet" "~" (id 3) (at 123.19 97.79 0)
+      (effects (font (size 1.27 1.27)) hide)
+    )
+    (property "MPN" "CC0603JRX7R8BB104" (id 4) (at 123.19 97.79 0)
       (effects (font (size 1.27 1.27)) hide)
     )
@@
   (symbol (lib_id "power:GND") (at 163.83 102.87 0) (unit 1)
     (in_bom yes) (on_board yes) (fields_autoplaced)
-    (property "Reference" "#PWR?" (id 0) (at 163.83 109.22 0)
+    (property "Reference" "#PWR024" (id 0) (at 163.83 109.22 0)
       (effects (font (size 1.27 1.27)) hide)
     )
@@
   (symbol (lib_id "power:GND") (at 123.19 102.87 0) (unit 1)
     (in_bom yes) (on_board yes) (fields_autoplaced)
-    (property "Reference" "#PWR?" (id 0) (at 123.19 109.22 0)
+    (property "Reference" "#PWR023" (id 0) (at 123.19 109.22 0)
       (effects (font (size 1.27 1.27)) hide)
     )

Commit message: So many updates
Parts:
- added C28: 0.1uF, Capacitor_SMD:C_0402_1005Metric, symbol Device:C_Small
- added C29: 680pF, Capacitor_SMD:C_0402_1005Metric, symbol Device:C_Small
- added R39: 100, Resistor_SMD:R_0402_1005Metric, symbol Device:R_Small_US
- added U15: TMP236AQDBZRQ1, Package_TO_SOT_SMD:SC-59, symbol ProjectSymbols:TMP236AQDBZRQ1
- C12: footprint Capacitor_SMD:C_0603_1608Metric -> Capacitor_SMD:C_0402_1005Metric; MPN CC0603JRX7R8BB104 -> CC0402KPX7R8BB104
- C13: footprint Capacitor_SMD:C_0603_1608Metric -> Capacitor_SMD:C_0402_1005Metric; MPN CC0603JRNPO8BN681 -> CC0402JRNPO9BN681
- R13: footprint Resistor_SMD:R_0603_1608Metric -> Resistor_SMD:R_0402_1005Metric; MPN RC0603FR-07100RL -> RC0402JR-07100RL
Connections:
- net +3V3: now also R39.1
- net GND: now also C28.1, C29.1, U15.3 (GND)
- net TEMP_VSENSE renamed LTEMP_VSENSE
- new net: C28.2, R39.2, U15.1 (VDD)
- new net RTEMP_VSENSE: C29.2, U15.2 (VOUT)
Changed lines of the file:
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@@
 (kicad_sch (version 20211123) (generator eeschema)
   (paper "A4")
+  (junction (at 123.19 113.03) (diameter 0) (color 0 0 0 0)
+  )
   (junction (at 123.19 92.71) (diameter 0) (color 0 0 0 0)
   )
   (junction (at 172.72 92.71) (diameter 0) (color 0 0 0 0)
   )
+  (junction (at 172.72 113.03) (diameter 0) (color 0 0 0 0)
+  )
   (wire (pts (xy 172.72 92.71) (xy 187.96 92.71))
     (stroke (width 0) (type default) (color 0 0 0 0))
   )
+  (wire (pts (xy 172.72 120.65) (xy 172.72 123.19))
+    (stroke (width 0) (type default) (color 0 0 0 0))
+  )
   (wire (pts (xy 123.19 92.71) (xy 119.38 92.71))
     (stroke (width 0) (type default) (color 0 0 0 0))
   )
+  (wire (pts (xy 163.83 123.19) (xy 163.83 118.11))
+    (stroke (width 0) (type default) (color 0 0 0 0))
+  )
+  (wire (pts (xy 172.72 113.03) (xy 160.02 113.03))
+    (stroke (width 0) (type default) (color 0 0 0 0))
+  )
+  (wire (pts (xy 163.83 118.11) (xy 160.02 118.11))
+    (stroke (width 0) (type default) (color 0 0 0 0))
+  )
+  (wire (pts (xy 110.49 113.03) (xy 114.3 113.03))
+    (stroke (width 0) (type default) (color 0 0 0 0))
+  )
   (wire (pts (xy 172.72 95.25) (xy 172.72 92.71))
     (stroke (width 0) (type default) (color 0 0 0 0))
@@
     (stroke (width 0) (type default) (color 0 0 0 0))
   )
+  (wire (pts (xy 123.19 120.65) (xy 123.19 123.19))
+    (stroke (width 0) (type default) (color 0 0 0 0))
+  )
   (wire (pts (xy 110.49 92.71) (xy 114.3 92.71))
     (stroke (width 0) (type default) (color 0 0 0 0))
@@
     (stroke (width 0) (type default) (color 0 0 0 0))
   )
+  (wire (pts (xy 123.19 113.03) (xy 140.97 113.03))
+    (stroke (width 0) (type default) (color 0 0 0 0))
+  )
+  (wire (pts (xy 172.72 113.03) (xy 187.96 113.03))
+    (stroke (width 0) (type default) (color 0 0 0 0))
+  )
+  (wire (pts (xy 123.19 115.57) (xy 123.19 113.03))
+    (stroke (width 0) (type default) (color 0 0 0 0))
+  )
   (wire (pts (xy 123.19 92.71) (xy 140.97 92.71))
     (stroke (width 0) (type default) (color 0 0 0 0))
@@
     (stroke (width 0) (type default) (color 0 0 0 0))
   )
+  (wire (pts (xy 172.72 115.57) (xy 172.72 113.03))
+    (stroke (width 0) (type default) (color 0 0 0 0))
+  )
   (wire (pts (xy 172.72 92.71) (xy 160.02 92.71))
     (stroke (width 0) (type default) (color 0 0 0 0))
+  )
+  (wire (pts (xy 123.19 113.03) (xy 119.38 113.03))
+    (stroke (width 0) (type default) (color 0 0 0 0))
+  )
+  (hierarchical_label "RTEMP_VSENSE" (shape output) (at 187.96 113.03 0)
+    (effects (font (size 1.27 1.27)) (justify left))
   )
   (hierarchical_label "+3V3" (shape input) (at 110.49 92.71 180)
     (effects (font (size 1.27 1.27)) (justify right))
   )
-  (hierarchical_label "TEMP_VSENSE" (shape output) (at 187.96 92.71 0)
+  (hierarchical_label "LTEMP_VSENSE" (shape output) (at 187.96 92.71 0)
     (effects (font (size 1.27 1.27)) (justify left))
+  )
+  (hierarchical_label "+3V3" (shape input) (at 110.49 113.03 180)
+    (effects (font (size 1.27 1.27)) (justify right))
   )
   (symbol (lib_id "ProjectSymbols:TMP236AQDBZRQ1") (at 149.86 96.52 0) (unit 1)
@@
     (property "Reference" "R13" (id 0) (at 116.84 86.36 90))
     (property "Value" "100" (id 1) (at 116.84 88.9 90))
-    (property "Footprint" "Resistor_SMD:R_0603_1608Metric" (id 2) (at 116.84 92.71 0)
+    (property "Footprint" "Resistor_SMD:R_0402_1005Metric" (id 2) (at 116.84 92.71 0)
       (effects (font (size 1.27 1.27)) hide)
     )
@@
       (effects (font (size 1.27 1.27)) hide)
     )
-    (property "MPN" "RC0603FR-07100RL" (id 4) (at 116.84 92.71 0)
+    (property "MPN" "RC0402JR-07100RL" (id 4) (at 116.84 92.71 0)
       (effects (font (size 1.27 1.27)) hide)
     )
@@
     (pin "1")
   )
+  (symbol (lib_id "Device:R_Small_US") (at 116.84 113.03 90) (unit 1)
+    (in_bom yes) (on_board yes) (fields_autoplaced)
+    (property "Reference" "R39" (id 0) (at 116.84 106.68 90))
+    (property "Value" "100" (id 1) (at 116.84 109.22 90))
+    (property "Footprint" "Resistor_SMD:R_0402_1005Metric" (id 2) (at 116.84 113.03 0)
+      (effects (font (size 1.27 1.27)) hide)
+    )
+    (property "Datasheet" "~" (id 3) (at 116.84 113.03 0)
+      (effects (font (size 1.27 1.27)) hide)
+    )
+    (property "MPN" "RC0402JR-07100RL" (id 4) (at 116.84 113.03 0)
+      (effects (font (size 1.27 1.27)) hide)
+    )
+    (pin "1")
+    (pin "2")
+  )
   (symbol (lib_id "Device:C_Small") (at 172.72 97.79 180) (unit 1)
     (in_bom yes) (on_board yes) (fields_autoplaced)
@@
       (effects (font (size 1.27 1.27)) (justify right))
     )
-    (property "Footprint" "Capacitor_SMD:C_0603_1608Metric" (id 2) (at 172.72 97.79 0)
+    (property "Footprint" "Capacitor_SMD:C_0402_1005Metric" (id 2) (at 172.72 97.79 0)
       (effects (font (size 1.27 1.27)) hide)
     )
@@
       (effects (font (size 1.27 1.27)) hide)
     )
-    (property "MPN" "CC0603JRNPO8BN681" (id 4) (at 172.72 97.79 0)
-      (effects (font (size 1.27 1.27)) hide)
-    )
-    (pin "1")
-    (pin "2")
+    (property "MPN" "CC0402JRNPO9BN681" (id 4) (at 172.72 97.79 0)
+      (effects (font (size 1.27 1.27)) hide)
+    )
+    (pin "1")
+    (pin "2")
+  )
+  (symbol (lib_id "power:GND") (at 123.19 123.19 0) (unit 1)
+    (in_bom yes) (on_board yes) (fields_autoplaced)
+    (property "Reference" "#PWR049" (id 0) (at 123.19 129.54 0)
+      (effects (font (size 1.27 1.27)) hide)
+    )
+    (property "Value" "GND" (id 1) (at 123.19 128.27 0)
+      (effects (font (size 1.27 1.27)) hide)
+    )
+    (property "Footprint" "" (id 2) (at 123.19 123.19 0)
+      (effects (font (size 1.27 1.27)) hide)
+    )
+    (property "Datasheet" "" (id 3) (at 123.19 123.19 0)
+      (effects (font (size 1.27 1.27)) hide)
+    )
+    (pin "1")
+  )
+  (symbol (lib_id "power:GND") (at 172.72 123.19 0) (unit 1)
+    (in_bom yes) (on_board yes) (fields_autoplaced)
+    (property "Reference" "#PWR051" (id 0) (at 172.72 129.54 0)
+      (effects (font (size 1.27 1.27)) hide)
+    )
+    (property "Value" "GND" (id 1) (at 172.72 128.27 0)
+      (effects (font (size 1.27 1.27)) hide)
+    )
+    (property "Footprint" "" (id 2) (at 172.72 123.19 0)
+      (effects (font (size 1.27 1.27)) hide)
+    )
+    (property "Datasheet" "" (id 3) (at 172.72 123.19 0)
+      (effects (font (size 1.27 1.27)) hide)
+    )
+    (pin "1")
+  )
+  (symbol (lib_id "Device:C_Small") (at 123.19 118.11 180) (unit 1)
+    (in_bom yes) (on_board yes) (fields_autoplaced)
+    (property "Reference" "C28" (id 0) (at 125.73 116.8335 0)
+      (effects (font (size 1.27 1.27)) (justify right))
+    )
+    (property "Value" "0.1uF" (id 1) (at 125.73 119.3735 0)
+      (effects (font (size 1.27 1.27)) (justify right))
+    )
+    (property "Footprint" "Capacitor_SMD:C_0402_1005Metric" (id 2) (at 123.19 118.11 0)
+      (effects (font (size 1.27 1.27)) hide)
+    )
+    (property "Datasheet" "~" (id 3) (at 123.19 118.11 0)
+      (effects (font (size 1.27 1.27)) hide)
+    )
+    (property "MPN" "CC0402KPX7R8BB104" (id 4) (at 123.19 118.11 0)
+      (effects (font (size 1.27 1.27)) hide)
+    )
+    (pin "1")
+    (pin "2")
+  )
+  (symbol (lib_id "power:GND") (at 163.83 123.19 0) (unit 1)
+    (in_bom yes) (on_board yes) (fields_autoplaced)
+    (property "Reference" "#PWR050" (id 0) (at 163.83 129.54 0)
+      (effects (font (size 1.27 1.27)) hide)
+    )
+    (property "Value" "GND" (id 1) (at 163.83 128.27 0)
+      (effects (font (size 1.27 1.27)) hide)
+    )
+    (property "Footprint" "" (id 2) (at 163.83 123.19 0)
+      (effects (font (size 1.27 1.27)) hide)
+    )
+    (property "Datasheet" "" (id 3) (at 163.83 123.19 0)
+      (effects (font (size 1.27 1.27)) hide)
+    )
+    (pin "1")
   )
   (symbol (lib_id "Device:C_Small") (at 123.19 97.79 180) (unit 1)
@@
       (effects (font (size 1.27 1.27)) (justify right))
     )
-    (property "Footprint" "Capacitor_SMD:C_0603_1608Metric" (id 2) (at 123.19 97.79 0)
+    (property "Footprint" "Capacitor_SMD:C_0402_1005Metric" (id 2) (at 123.19 97.79 0)
       (effects (font (size 1.27 1.27)) hide)
     )
@@
       (effects (font (size 1.27 1.27)) hide)
     )
-    (property "MPN" "CC0603JRX7R8BB104" (id 4) (at 123.19 97.79 0)
+    (property "MPN" "CC0402KPX7R8BB104" (id 4) (at 123.19 97.79 0)
+      (effects (font (size 1.27 1.27)) hide)
+    )
+    (pin "1")
+    (pin "2")
+  )
+  (symbol (lib_id "Device:C_Small") (at 172.72 118.11 180) (unit 1)
+    (in_bom yes) (on_board yes) (fields_autoplaced)
+    (property "Reference" "C29" (id 0) (at 175.26 116.8335 0)
+      (effects (font (size 1.27 1.27)) (justify right))
+    )
+    (property "Value" "680pF" (id 1) (at 175.26 119.3735 0)
+      (effects (font (size 1.27 1.27)) (justify right))
+    )
+    (property "Footprint" "Capacitor_SMD:C_0402_1005Metric" (id 2) (at 172.72 118.11 0)
+      (effects (font (size 1.27 1.27)) hide)
+    )
+    (property "Datasheet" "~" (id 3) (at 172.72 118.11 0)
+      (effects (font (size 1.27 1.27)) hide)
+    )
+    (property "MPN" "CC0402JRNPO9BN681" (id 4) (at 172.72 118.11 0)
       (effects (font (size 1.27 1.27)) hide)
     )
@@
     (pin "1")
   )
+  (symbol (lib_id "ProjectSymbols:TMP236AQDBZRQ1") (at 149.86 116.84 0) (unit 1)
+    (in_bom yes) (on_board yes) (fields_autoplaced)
+    (property "Reference" "U15" (id 0) (at 150.495 106.68 0))
+    (property "Value" "TMP236AQDBZRQ1" (id 1) (at 150.495 109.22 0))
+    (property "Footprint" "Package_TO_SOT_SMD:SC-59" (id 2) (at 152.4 100.33 0)
+      (effects (font (size 1.27 1.27)) hide)
+    )
+    (property "Datasheet" "" (id 3) (at 152.4 100.33 0)
+      (effects (font (size 1.27 1.27)) hide)
+    )
+    (property "MPN" "TMP236AQDBZRQ1" (id 4) (at 149.86 116.84 0)
+      (effects (font (size 1.27 1.27)) hide)
+    )
+    (pin "1")
+    (pin "2")
+    (pin "3")
+  )
 )
