File: MotorController/USB.kicad_sch (KiCad schematic)
At the start: 0 parts

Commit message: Schematic Updates
Parts:
- added C?: 0.1uF, symbol Device:C_Small
- added C?: 1uF, symbol Device:C_Small
- added J?: USB_B_Micro, symbol Connector:USB_B_Micro
- added R? (x2): 0, symbol Device:R_Small_US
- added U?: TPD2E2U06DCKR, symbol ProjectSymbols:TPD2E2U06DCKR
- added U?: FT234XD-R, symbol ProjectSymbols:FT234XD-R
Connections:
- new net: J?.3 (D+), U?.1 (IO1), U?.1 (USBDM), U?.2 (IO2)
- new net: R?.2, U?.8 (~{RTS})
- new net: R?.1, U?.11 (~{CTS})
- new net: J?.2 (D-), U?.12 (USBDP)
- new net +3V3: C?.1, C?.1, U?.2 (~{RESET}), U?.3 (3V3OUT), U?.4 (VCC), U?.9 (VCCIO)
- new net +VUSB: J?.1 (VBUS)
- new net GND: C?.2, C?.2, J?.5 (GND), J?.6 (Shield), U?.13 (GND), U?.3 (GND), U?.5 (GND)
- new net RXD: U?.10 (RXD)
- new net TXD: U?.7 (TXD)
- new net ~{CTS}: R?.1
- new net ~{RTS}: R?.2
- no-connect marks 0 -> 2

Commit message: Updates
Parts:
- removed R? (x2): 0, symbol Device:R_Small_US
- C10: renamed from C?; footprint (none) -> Capacitor_SMD:C_0603_1608Metric; MPN (none) -> CC0603KRX5R8BB105
- C11: renamed from C?; footprint (none) -> Capacitor_SMD:C_0603_1608Metric; MPN (none) -> CC0603JRX7R8BB104
- J4: renamed from J?; footprint (none) -> Footprints:CUI_UJ2-MIBH-G-SMT-TR; MPN (none) -> UJ2-MIBH-G-SMT-TR
- U5: renamed from U?; footprint (none) -> Package_TO_SOT_SMD:SOT-323_SC-70; MPN (none) -> TPD2E2U06DCKR
- U6: renamed from U?; footprint (none) -> Package_DFN_QFN:DFN-12-1EP_3x3mm_P0.5mm_EP1.6x2.5mm; MPN (none) -> FT234XD-R
Connections:
- no-connect marks 2 -> 4
Changed lines of the file:
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@@
   (no_connect (at 71.12 76.2))
   (no_connect (at 140.97 72.39))
-  (wire (pts (xy 140.97 68.58) (xy 156.21 68.58))
-    (stroke (width 0) (type default) (color 0 0 0 0))
-  )
+  (no_connect (at 140.97 66.04))
+  (no_connect (at 140.97 68.58))
   (wire (pts (xy 63.5 83.82) (xy 63.5 86.36))
     (stroke (width 0) (type default) (color 0 0 0 0))
@@
     (stroke (width 0) (type default) (color 0 0 0 0))
   )
-  (wire (pts (xy 140.97 66.04) (xy 156.21 66.04))
-    (stroke (width 0) (type default) (color 0 0 0 0))
-  )
   (wire (pts (xy 60.96 81.28) (xy 60.96 83.82))
     (stroke (width 0) (type default) (color 0 0 0 0))
@@
     (stroke (width 0) (type default) (color 0 0 0 0))
   )
-  (wire (pts (xy 161.29 68.58) (xy 167.64 68.58))
-    (stroke (width 0) (type default) (color 0 0 0 0))
-  )
   (wire (pts (xy 86.36 81.28) (xy 83.82 81.28))
     (stroke (width 0) (type default) (color 0 0 0 0))
@@
     (stroke (width 0) (type default) (color 0 0 0 0))
   )
-  (wire (pts (xy 161.29 66.04) (xy 167.64 66.04))
-    (stroke (width 0) (type default) (color 0 0 0 0))
-  )
   (wire (pts (xy 99.06 38.1) (xy 109.22 38.1))
     (stroke (width 0) (type default) (color 0 0 0 0))
@@
   (wire (pts (xy 116.84 58.42) (xy 116.84 60.96))
     (stroke (width 0) (type default) (color 0 0 0 0))
-  )
-  (hierarchical_label "~{RTS}" (shape output) (at 167.64 66.04 0)
-    (effects (font (size 1.27 1.27)) (justify left))
   )
   (hierarchical_label "RXD" (shape input) (at 144.78 60.96 0)
@@
     (effects (font (size 1.27 1.27)) (justify left))
   )
-  (hierarchical_label "~{CTS}" (shape input) (at 167.64 68.58 0)
-    (effects (font (size 1.27 1.27)) (justify left))
-  )
   (hierarchical_label "TXD" (shape output) (at 144.78 58.42 0)
     (effects (font (size 1.27 1.27)) (justify left))
@@
   (symbol (lib_id "power:GND") (at 93.98 92.71 0) (unit 1)
     (in_bom yes) (on_board yes) (fields_autoplaced)
-    (property "Reference" "#PWR?" (id 0) (at 93.98 99.06 0)
+    (property "Reference" "#PWR019" (id 0) (at 93.98 99.06 0)
       (effects (font (size 1.27 1.27)) hide)
     )
@@
   (symbol (lib_id "power:GND") (at 99.06 48.26 0) (unit 1)
     (in_bom yes) (on_board yes) (fields_autoplaced)
-    (property "Reference" "#PWR?" (id 0) (at 99.06 54.61 0)
+    (property "Reference" "#PWR020" (id 0) (at 99.06 54.61 0)
       (effects (font (size 1.27 1.27)) hide)
     )
@@
   (symbol (lib_id "power:GND") (at 143.51 81.28 0) (unit 1)
     (in_bom yes) (on_board yes) (fields_autoplaced)
-    (property "Reference" "#PWR?" (id 0) (at 143.51 87.63 0)
+    (property "Reference" "#PWR022" (id 0) (at 143.51 87.63 0)
       (effects (font (size 1.27 1.27)) hide)
     )
@@
   (symbol (lib_id "power:GND") (at 63.5 86.36 0) (unit 1)
     (in_bom yes) (on_board yes) (fields_autoplaced)
-    (property "Reference" "#PWR?" (id 0) (at 63.5 92.71 0)
+    (property "Reference" "#PWR018" (id 0) (at 63.5 92.71 0)
       (effects (font (size 1.27 1.27)) hide)
     )
@@
   (symbol (lib_id "ProjectSymbols:TPD2E2U06DCKR") (at 93.98 85.09 0) (unit 1)
     (in_bom yes) (on_board yes) (fields_autoplaced)
-    (property "Reference" "U?" (id 0) (at 93.98 74.93 0))
+    (property "Reference" "U5" (id 0) (at 93.98 74.93 0))
     (property "Value" "TPD2E2U06DCKR" (id 1) (at 93.98 77.47 0))
-    (property "Footprint" "" (id 2) (at 93.98 73.66 0)
+    (property "Footprint" "Package_TO_SOT_SMD:SOT-323_SC-70" (id 2) (at 93.98 73.66 0)
       (effects (font (size 1.27 1.27)) hide)
     )
     (property "Datasheet" "" (id 3) (at 93.98 73.66 0)
+      (effects (font (size 1.27 1.27)) hide)
+    )
+    (property "MPN" "TPD2E2U06DCKR" (id 4) (at 93.98 85.09 0)
       (effects (font (size 1.27 1.27)) hide)
     )
@@
     (pin "3")
   )
-  (symbol (lib_id "Device:R_Small_US") (at 158.75 68.58 270) (unit 1)
-    (in_bom yes) (on_board yes)
-    (property "Reference" "R?" (id 0) (at 158.75 73.66 90))
-    (property "Value" "0" (id 1) (at 158.75 71.12 90))
-    (property "Footprint" "" (id 2) (at 158.75 68.58 0)
-      (effects (font (size 1.27 1.27)) hide)
-    )
-    (property "Datasheet" "~" (id 3) (at 158.75 68.58 0)
-      (effects (font (size 1.27 1.27)) hide)
-    )
-    (pin "1")
-    (pin "2")
-  )
   (symbol (lib_id "ProjectSymbols:FT234XD-R") (at 130.81 68.58 0) (unit 1)
     (in_bom yes) (on_board yes) (fields_autoplaced)
-    (property "Reference" "U?" (id 0) (at 130.175 52.07 0))
+    (property "Reference" "U6" (id 0) (at 130.175 52.07 0))
     (property "Value" "FT234XD-R" (id 1) (at 130.175 54.61 0))
-    (property "Footprint" "" (id 2) (at 130.81 54.61 0)
+    (property "Footprint" "Package_DFN_QFN:DFN-12-1EP_3x3mm_P0.5mm_EP1.6x2.5mm" (id 2) (at 130.81 54.61 0)
       (effects (font (size 1.27 1.27)) hide)
     )
     (property "Datasheet" "" (id 3) (at 130.81 54.61 0)
+      (effects (font (size 1.27 1.27)) hide)
+    )
+    (property "MPN" "FT234XD-R" (id 4) (at 130.81 68.58 0)
       (effects (font (size 1.27 1.27)) hide)
     )
@@
   (symbol (lib_id "Device:C_Small") (at 109.22 43.18 0) (unit 1)
     (in_bom yes) (on_board yes) (fields_autoplaced)
-    (property "Reference" "C?" (id 0) (at 111.76 41.9162 0)
+    (property "Reference" "C11" (id 0) (at 111.76 41.9162 0)
       (effects (font (size 1.27 1.27)) (justify left))
     )
@@
       (effects (font (size 1.27 1.27)) (justify left))
     )
-    (property "Footprint" "" (id 2) (at 109.22 43.18 0)
+    (property "Footprint" "Capacitor_SMD:C_0603_1608Metric" (id 2) (at 109.22 43.18 0)
       (effects (font (size 1.27 1.27)) hide)
     )
@@
       (effects (font (size 1.27 1.27)) hide)
     )
+    (property "MPN" "CC0603JRX7R8BB104" (id 4) (at 109.22 43.18 0)
+      (effects (font (size 1.27 1.27)) hide)
+    )
     (pin "1")
     (pin "2")
   )
-  (symbol (lib_id "Device:R_Small_US") (at 158.75 66.04 90) (unit 1)
-    (in_bom yes) (on_board yes) (fields_autoplaced)
-    (property "Reference" "R?" (id 0) (at 158.75 59.69 90))
-    (property "Value" "0" (id 1) (at 158.75 62.23 90))
-    (property "Footprint" "" (id 2) (at 158.75 66.04 0)
-      (effects (font (size 1.27 1.27)) hide)
-    )
-    (property "Datasheet" "~" (id 3) (at 158.75 66.04 0)
-      (effects (font (size 1.27 1.27)) hide)
-    )
-    (pin "1")
-    (pin "2")
-  )
   (symbol (lib_id "Connector:USB_B_Micro") (at 63.5 71.12 0) (unit 1)
     (in_bom yes) (on_board yes) (fields_autoplaced)
-    (property "Reference" "J?" (id 0) (at 63.5 58.42 0))
+    (property "Reference" "J4" (id 0) (at 63.5 58.42 0))
     (property "Value" "USB_B_Micro" (id 1) (at 63.5 60.96 0))
-    (property "Footprint" "" (id 2) (at 67.31 72.39 0)
+    (property "Footprint" "Footprints:CUI_UJ2-MIBH-G-SMT-TR" (id 2) (at 67.31 72.39 0)
       (effects (font (size 1.27 1.27)) hide)
     )
     (property "Datasheet" "~" (id 3) (at 67.31 72.39 0)
+      (effects (font (size 1.27 1.27)) hide)
+    )
+    (property "MPN" "UJ2-MIBH-G-SMT-TR" (id 4) (at 63.5 71.12 0)
       (effects (font (size 1.27 1.27)) hide)
     )
@@
   (symbol (lib_id "power:GND") (at 109.22 48.26 0) (unit 1)
     (in_bom yes) (on_board yes) (fields_autoplaced)
-    (property "Reference" "#PWR?" (id 0) (at 109.22 54.61 0)
+    (property "Reference" "#PWR021" (id 0) (at 109.22 54.61 0)
       (effects (font (size 1.27 1.27)) hide)
     )
@@
   (symbol (lib_id "Device:C_Small") (at 99.06 43.18 0) (unit 1)
     (in_bom yes) (on_board yes) (fields_autoplaced)
-    (property "Reference" "C?" (id 0) (at 101.6 41.9162 0)
+    (property "Reference" "C10" (id 0) (at 101.6 41.9162 0)
       (effects (font (size 1.27 1.27)) (justify left))
     )
@@
       (effects (font (size 1.27 1.27)) (justify left))
     )
-    (property "Footprint" "" (id 2) (at 99.06 43.18 0)
+    (property "Footprint" "Capacitor_SMD:C_0603_1608Metric" (id 2) (at 99.06 43.18 0)
       (effects (font (size 1.27 1.27)) hide)
     )
@@
       (effects (font (size 1.27 1.27)) hide)
     )
+    (property "MPN" "CC0603KRX5R8BB105" (id 4) (at 99.06 43.18 0)
+      (effects (font (size 1.27 1.27)) hide)
+    )

Commit message: So many updates
Parts:
- C10: footprint Capacitor_SMD:C_0603_1608Metric -> Capacitor_SMD:C_0402_1005Metric; MPN CC0603KRX5R8BB105 -> CC0402KRX5R8BB105
- C11: footprint Capacitor_SMD:C_0603_1608Metric -> Capacitor_SMD:C_0402_1005Metric; MPN CC0603JRX7R8BB104 -> CC0402KPX7R8BB104
Changed lines of the file:
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@@
       (effects (font (size 1.27 1.27)) (justify left))
     )
-    (property "Footprint" "Capacitor_SMD:C_0603_1608Metric" (id 2) (at 109.22 43.18 0)
+    (property "Footprint" "Capacitor_SMD:C_0402_1005Metric" (id 2) (at 109.22 43.18 0)
       (effects (font (size 1.27 1.27)) hide)
     )
@@
       (effects (font (size 1.27 1.27)) hide)
     )
-    (property "MPN" "CC0603JRX7R8BB104" (id 4) (at 109.22 43.18 0)
+    (property "MPN" "CC0402KPX7R8BB104" (id 4) (at 109.22 43.18 0)
       (effects (font (size 1.27 1.27)) hide)
     )
@@
       (effects (font (size 1.27 1.27)) (justify left))
     )
-    (property "Footprint" "Capacitor_SMD:C_0603_1608Metric" (id 2) (at 99.06 43.18 0)
+    (property "Footprint" "Capacitor_SMD:C_0402_1005Metric" (id 2) (at 99.06 43.18 0)
       (effects (font (size 1.27 1.27)) hide)
     )
@@
       (effects (font (size 1.27 1.27)) hide)
     )
-    (property "MPN" "CC0603KRX5R8BB105" (id 4) (at 99.06 43.18 0)
+    (property "MPN" "CC0402KRX5R8BB105" (id 4) (at 99.06 43.18 0)
       (effects (font (size 1.27 1.27)) hide)
     )

Commit message: my god
my god
Connections:
- net DP: now reaches J4.3 (D+), U5.1 (IO1), U6.1 (USBDM)
- net DP: no longer U5.2 (IO2)
- net DN: now reaches J4.2 (D-), U6.12 (USBDP)
- net DN: now also U5.2 (IO2)
Changed lines of the file:
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@@
   (junction (at 63.5 83.82) (diameter 0) (color 0 0 0 0)
-  )
-  (junction (at 83.82 71.12) (diameter 0) (color 0 0 0 0)
   )
   (junction (at 99.06 38.1) (diameter 0) (color 0 0 0 0)
@@
   (junction (at 116.84 63.5) (diameter 0) (color 0 0 0 0)
   )
+  (junction (at 83.82 71.12) (diameter 0) (color 0 0 0 0)
+  )
   (junction (at 143.51 78.74) (diameter 0) (color 0 0 0 0)
   )
-  (junction (at 104.14 71.12) (diameter 0) (color 0 0 0 0)
+  (junction (at 104.14 73.66) (diameter 0) (color 0 0 0 0)
   )
   (junction (at 116.84 58.42) (diameter 0) (color 0 0 0 0)
@@
   (no_connect (at 140.97 66.04))
   (no_connect (at 140.97 68.58))
+  (wire (pts (xy 83.82 71.12) (xy 119.38 71.12))
+    (stroke (width 0) (type default) (color 0 0 0 0))
+  )
   (wire (pts (xy 63.5 83.82) (xy 63.5 86.36))
     (stroke (width 0) (type default) (color 0 0 0 0))
   )
   (wire (pts (xy 116.84 63.5) (xy 119.38 63.5))
+    (stroke (width 0) (type default) (color 0 0 0 0))
+  )
+  (wire (pts (xy 104.14 73.66) (xy 119.38 73.66))
     (stroke (width 0) (type default) (color 0 0 0 0))
   )
@@
     (stroke (width 0) (type default) (color 0 0 0 0))
   )
-  (wire (pts (xy 104.14 81.28) (xy 104.14 71.12))
-    (stroke (width 0) (type default) (color 0 0 0 0))
-  )
   (wire (pts (xy 101.6 81.28) (xy 104.14 81.28))
     (stroke (width 0) (type default) (color 0 0 0 0))
   )
   (wire (pts (xy 140.97 78.74) (xy 143.51 78.74))
-    (stroke (width 0) (type default) (color 0 0 0 0))
-  )
-  (wire (pts (xy 83.82 81.28) (xy 83.82 71.12))
     (stroke (width 0) (type default) (color 0 0 0 0))
   )
@@
   )
   (wire (pts (xy 116.84 38.1) (xy 116.84 58.42))
-    (stroke (width 0) (type default) (color 0 0 0 0))
-  )
-  (wire (pts (xy 71.12 71.12) (xy 83.82 71.12))
-    (stroke (width 0) (type default) (color 0 0 0 0))
-  )
-  (wire (pts (xy 83.82 71.12) (xy 104.14 71.12))
     (stroke (width 0) (type default) (color 0 0 0 0))
   )
@@
     (stroke (width 0) (type default) (color 0 0 0 0))
   )
+  (wire (pts (xy 83.82 71.12) (xy 83.82 81.28))
+    (stroke (width 0) (type default) (color 0 0 0 0))
+  )
   (wire (pts (xy 86.36 81.28) (xy 83.82 81.28))
     (stroke (width 0) (type default) (color 0 0 0 0))
@@
   )
   (wire (pts (xy 116.84 60.96) (xy 116.84 63.5))
+    (stroke (width 0) (type default) (color 0 0 0 0))
+  )
+  (wire (pts (xy 104.14 73.66) (xy 104.14 81.28))
     (stroke (width 0) (type default) (color 0 0 0 0))
   )
@@
     (stroke (width 0) (type default) (color 0 0 0 0))
   )
-  (wire (pts (xy 71.12 73.66) (xy 119.38 73.66))
+  (wire (pts (xy 71.12 73.66) (xy 104.14 73.66))
     (stroke (width 0) (type default) (color 0 0 0 0))
   )
-  (wire (pts (xy 104.14 71.12) (xy 119.38 71.12))
+  (wire (pts (xy 71.12 71.12) (xy 83.82 71.12))
     (stroke (width 0) (type default) (color 0 0 0 0))
   )
@@
     (stroke (width 0) (type default) (color 0 0 0 0))
   )
+  (label "DP" (at 87.63 71.12 0)
+    (effects (font (size 1.27 1.27)) (justify left bottom))
+  )
+  (label "DN" (at 87.63 73.66 0)
+    (effects (font (size 1.27 1.27)) (justify left bottom))
+  )
   (hierarchical_label "RXD" (shape input) (at 144.78 60.96 0)
