File: MotorController/LMOTOR.kicad_sch (KiCad schematic)
At the start: 0 parts

Commit message: Updates
Updates
Parts:
- added C? (x2): 1uF, symbol Device:C_Small
- added C? (x2): 40nF, symbol Device:C_Small
- added D? (x4): D_Small_Filled, symbol Device:D_Small_Filled
- added M?: Motor_DC, symbol Motor:Motor_DC
- added Q? (x4): Q_NMOS_GDS, symbol Device:Q_NMOS_GDS
- added R? (x2): DNU, symbol Device:R_Small_US
- added R?: 0, symbol Device:R_Small_US
- added U? (x2): 2EDL8024GX, symbol ProjectSymbols:2EDL8024GX
Connections:
- new net: Q?.1 (G), U?.8 (LO) (x2)
- new net: C?.2, D?.1 (K), D?.2 (A), M?.1 (+), Q?.2 (D), Q?.3 (S), U?.4 (HS)
- new net: C?.2, D?.1 (K), D?.2 (A), M?.2 (-), Q?.2 (D), Q?.3 (S), U?.4 (HS)
- new net: Q?.1 (G), U?.3 (HO) (x2)
- new net +3V3: R?.1
- new net +5V: R?.1
- new net +BATT: D?.1 (K), D?.1 (K), Q?.2 (D), Q?.2 (D), R?.1
- new net +VDD: C?.1, C?.1, R?.2, R?.2, R?.2, U?.1 (VDD), U?.1 (VDD)
- new net GND: C?.2, C?.2, D?.2 (A), D?.2 (A), Q?.3 (S), Q?.3 (S), U?.7 (VSS), U?.7 (VSS), U?.9 (VSS), U?.9 (VSS)
- new net LBOOTSTRAP: C?.1, U?.2 (HB)
- new net LMOTOR_BACKWARDS: U?.5 (HI), U?.6 (LI)
- new net LMOTOR_FORWARD: U?.5 (HI), U?.6 (LI)
- new net RBOOTSTRAP: C?.1, U?.2 (HB)

Commit message: More updates
Parts:
- added C?: 1000uF, symbol Device:C_Small
- added D? (x4): D_Small_Filled, symbol Device:D_Small_Filled
- added R? (x4): 2, symbol Device:R_Small_US
Connections:
- net +BATT: now also C?.1
- net GND: now also C?.2
- net at Q?.1 (G): now also D?.2 (A), R?.2; no longer U?.8 (LO)
- net at Q?.1 (G): now also D?.2 (A), R?.1; no longer U?.3 (HO) (x2)
- net at U?.8 (LO): now also D?.1 (K), R?.1; no longer Q?.1 (G)
- new net: D?.1 (K), R?.2, U?.3 (HO) (x2)
- new net: D?.1 (K), R?.1, U?.8 (LO)
- new net: D?.2 (A), Q?.1 (G), R?.2
Other:
- moved on the sheet: Q?

Commit message: Updates
Parts:
- C15, C19: renamed from C?; footprint (none) -> Capacitor_SMD:C_0603_1608Metric; MPN (none) -> CC0603KRX5R8BB105
- C16, C18: renamed from C?; footprint (none) -> Capacitor_SMD:C_0603_1608Metric; MPN (none) -> CC0603KRX7R8BB393
- C17: renamed from C?; value 1000uF -> 330uF; footprint (none) -> Capacitor_SMD:CP_Elec_10x10; MPN (none) -> A771MS337M1VLAS014
- D10, D11, D4, D5, D6, D7, D8, D9: renamed from D?; MPN (none) -> S1A-13-F
- M1: renamed from M?; footprint (none) -> Connector_PinHeader_2.54mm:PinHeader_1x02_P2.54mm_Vertical
- Q1, Q2, Q3, Q4: renamed from Q?; footprint (none) -> Footprints:TRANS_SSM6K513NU-LF; MPN (none) -> FDD8447L
- R14, R15, R16: renamed from R?; footprint (none) -> Resistor_SMD:R_0603_1608Metric; MPN (none) -> RC0603FR-070RL
- R17, R18, R19, R20: renamed from R?; footprint (none) -> Resistor_SMD:R_0603_1608Metric; MPN (none) -> RC0603FR-072RL
- U10, U9: renamed from U?; footprint (none) -> Package_DFN_QFN:DFN-8-1EP_4x4mm_P0.8mm_EP2.3x3.24mm; MPN (none) -> 2EDL8024GX

Commit message: Changes
Changes
Parts:
- removed D10, D11, D4: D_Small_Filled, symbol Device:D_Small_Filled
- removed Q1, Q2, Q3, Q4: Q_NMOS_GDS, Footprints:TRANS_SSM6K513NU-LF, symbol Device:Q_NMOS_GDS
- added D? (x3): D_Small_Filled, Diode_SMD:D_SOD-323, symbol Device:D_Small_Filled
- added Q1, Q2, Q3, Q4: SSM6K513NU-LF, Footprints:TRANS_SSM6K513NU-LF, symbol ProjectSymbols:SSM6K513NU-LF
- D5: footprint (none) -> Diode_SMD:D_SOD-323; MPN S1A-13-F -> NSR0530HT1G
- D6, D7, D8, D9: MPN S1A-13-F -> (none)
Connections:
- net +BATT: now also Q1.1, Q1.2, Q1.5, Q1.6, Q1.7, Q3.1, Q3.2, Q3.5, Q3.6, Q3.7
- net GND: now also Q2.4, Q2.8, Q4.4, Q4.8
- net at D5.2 (A), R18.2: now also Q2.3
- net at C16.2, D6.2 (A), D7.1 (K)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: now also Q1.4, Q1.8, Q2.1, Q2.2, Q2.5, Q2.6, Q2.7
- net at R17.1: now also D?.2 (A), Q1.3
- net at R17.2, U9.3 (HO): now also D?.1 (K)
- net at C18.2, D8.2 (A), D9.1 (K)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: now also Q3.4, Q3.8, Q4.1, Q4.2, Q4.5, Q4.6, Q4.7
- net at R19.1: now also D?.2 (A), Q3.3
- net at R20.1, U10.8 (LO): now also D?.1 (K)
- net at R20.2: now also D?.2 (A), Q4.3
- net at R19.2, U10.3 (HO): now also D?.1 (K)

Commit message: So many updates
Parts:
- removed D6, D7: D_Small_Filled, symbol Device:D_Small_Filled
- added D10, D11: D_Small_Filled, Footprints:TO-277B, symbol Device:D_Small_Filled
- C15, C19: footprint Capacitor_SMD:C_0603_1608Metric -> Capacitor_SMD:C_0402_1005Metric; MPN CC0603KRX5R8BB105 -> CC0402KRX5R8BB105
- C16, C18: value 40nF -> 33nF; footprint Capacitor_SMD:C_0603_1608Metric -> Capacitor_SMD:C_0402_1005Metric; MPN CC0603KRX7R8BB393 -> CC0402KRX7R9BB333
- C17: footprint Capacitor_SMD:CP_Elec_10x10 -> Connector_PinHeader_2.54mm:PinHeader_1x02_P2.54mm_Vertical; MPN A771MS337M1VLAS014 -> (none)
- D8, D9: footprint (none) -> Footprints:TO-277B; MPN (none) -> MBR1560S
- R14: footprint Resistor_SMD:R_0603_1608Metric -> Resistor_SMD:R_0402_1005Metric; MPN RC0603FR-070RL -> RC0402JR-070RL
- R15, R16: footprint Resistor_SMD:R_0603_1608Metric -> Resistor_SMD:R_0402_1005Metric; MPN RC0603FR-070RL -> RC0402JR-0710KL
- R17, R18, R19, R20: footprint Resistor_SMD:R_0603_1608Metric -> Resistor_SMD:R_0402_1005Metric; MPN RC0603FR-072RL -> RC0402FR-072RL
- gave numbers to parts that had none: 3
Connections:
- net +BATT: now also D10.1 (K)
- net GND: now also D11.2 (A)
- net at C18.2, M1.2 (-), Q3.4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: now also D10.2 (A), D11.1 (K); no longer D8.2 (A), D9.1 (K)
- net at C16.2, M1.1 (+), Q1.4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: now also D8.2 (A), D9.1 (K)

Commit message: my god
my god
Connections:
- net +VDD renamed +VDD_L
- net LBOOTSTRAP renamed LLBOOTSTRAP
- net RBOOTSTRAP renamed LRBOOTSTRAP
Changed lines of the file:
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@@
     (stroke (width 0) (type default) (color 0 0 0 0))
   )
-  (global_label "LBOOTSTRAP" (shape bidirectional) (at 107.95 35.56 180) (fields_autoplaced)
+  (global_label "LLBOOTSTRAP" (shape bidirectional) (at 107.95 35.56 180) (fields_autoplaced)
     (effects (font (size 1.27 1.27)) (justify right))
-    (property "Intersheet References" "${INTERSHEET_REFS}" (id 0) (at 93.8045 35.4806 0)
+    (property "Intersheet References" "${INTERSHEET_REFS}" (id 0) (at 92.7764 35.4806 0)
       (effects (font (size 1.27 1.27)) (justify right) hide)
     )
   )
-  (global_label "LBOOTSTRAP" (shape bidirectional) (at 78.74 64.77 180) (fields_autoplaced)
+  (global_label "LLBOOTSTRAP" (shape bidirectional) (at 78.74 64.77 180) (fields_autoplaced)
     (effects (font (size 1.27 1.27)) (justify right))
-    (property "Intersheet References" "${INTERSHEET_REFS}" (id 0) (at 64.5945 64.6906 0)
+    (property "Intersheet References" "${INTERSHEET_REFS}" (id 0) (at 63.5664 64.6906 0)
       (effects (font (size 1.27 1.27)) (justify right) hide)
     )
   )
-  (global_label "RBOOTSTRAP" (shape bidirectional) (at 203.2 35.56 0) (fields_autoplaced)
+  (global_label "LRBOOTSTRAP" (shape bidirectional) (at 203.2 35.56 0) (fields_autoplaced)
     (effects (font (size 1.27 1.27)) (justify left))
-    (property "Intersheet References" "${INTERSHEET_REFS}" (id 0) (at 217.5874 35.4806 0)
+    (property "Intersheet References" "${INTERSHEET_REFS}" (id 0) (at 218.6155 35.4806 0)
       (effects (font (size 1.27 1.27)) (justify left) hide)
     )
   )
-  (global_label "+VDD" (shape output) (at 48.26 33.02 0) (fields_autoplaced)
+  (global_label "+VDD_L" (shape output) (at 48.26 33.02 0) (fields_autoplaced)
     (effects (font (size 1.27 1.27)) (justify left))
-    (property "Intersheet References" "${INTERSHEET_REFS}" (id 0) (at 55.8741 32.9406 0)
+    (property "Intersheet References" "${INTERSHEET_REFS}" (id 0) (at 57.8698 32.9406 0)
       (effects (font (size 1.27 1.27)) (justify left) hide)
     )
   )
-  (global_label "RBOOTSTRAP" (shape bidirectional) (at 229.87 69.85 0) (fields_autoplaced)
+  (global_label "+VDD_L" (shape input) (at 269.24 52.07 0) (fields_autoplaced)
     (effects (font (size 1.27 1.27)) (justify left))
-    (property "Intersheet References" "${INTERSHEET_REFS}" (id 0) (at 244.2574 69.7706 0)
+    (property "Intersheet References" "${INTERSHEET_REFS}" (id 0) (at 278.8498 51.9906 0)
       (effects (font (size 1.27 1.27)) (justify left) hide)
     )
   )
-  (global_label "+VDD" (shape input) (at 43.18 46.99 180) (fields_autoplaced)
+  (global_label "LRBOOTSTRAP" (shape bidirectional) (at 229.87 69.85 0) (fields_autoplaced)
+    (effects (font (size 1.27 1.27)) (justify left))
+    (property "Intersheet References" "${INTERSHEET_REFS}" (id 0) (at 245.2855 69.7706 0)
+      (effects (font (size 1.27 1.27)) (justify left) hide)
+    )
+  )
+  (global_label "+VDD_L" (shape input) (at 43.18 46.99 180) (fields_autoplaced)
     (effects (font (size 1.27 1.27)) (justify right))
-    (property "Intersheet References" "${INTERSHEET_REFS}" (id 0) (at 35.5659 47.0694 0)
+    (property "Intersheet References" "${INTERSHEET_REFS}" (id 0) (at 33.5702 46.9106 0)
       (effects (font (size 1.27 1.27)) (justify right) hide)
     )
   )
-  (global_label "+VDD" (shape input) (at 269.24 52.07 0) (fields_autoplaced)
-    (effects (font (size 1.27 1.27)) (justify left))
-    (property "Intersheet References" "${INTERSHEET_REFS}" (id 0) (at 276.8541 52.1494 0)
-      (effects (font (size 1.27 1.27)) (justify left) hide)
-    )
-  )

Commit message: The monstrosity is almost done
The monstrosity is almost done
Parts:
- removed R14: 0, Resistor_SMD:R_0402_1005Metric, symbol Device:R_Small_US
Changed lines of the file:
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@@
-    (stroke (width 0) (type default) (color 0 0 0 0))
-  )
-  (wire (pts (xy 45.72 25.4) (xy 45.72 33.02))
     (stroke (width 0) (type default) (color 0 0 0 0))
   )
@@
     (stroke (width 0) (type default) (color 0 0 0 0))
   )
-  (wire (pts (xy 34.29 25.4) (xy 38.1 25.4))
-    (stroke (width 0) (type default) (color 0 0 0 0))
-  )
   (wire (pts (xy 184.15 36.83) (xy 184.15 40.64))
     (stroke (width 0) (type default) (color 0 0 0 0))
@@
   )
   (wire (pts (xy 34.29 33.02) (xy 38.1 33.02))
-    (stroke (width 0) (type default) (color 0 0 0 0))
-  )
-  (wire (pts (xy 43.18 25.4) (xy 45.72 25.4))
     (stroke (width 0) (type default) (color 0 0 0 0))
   )
@@
   )
   (hierarchical_label "+5V" (shape input) (at 34.29 33.02 180)
-    (effects (font (size 1.27 1.27)) (justify right))
-  )
-  (hierarchical_label "+3V3" (shape input) (at 34.29 25.4 180)
     (effects (font (size 1.27 1.27)) (justify right))
   )
@@
       (effects (font (size 1.27 1.27)) hide)
     )
-    (pin "1")
-    (pin "2")
-  )
-  (symbol (lib_id "Device:R_Small_US") (at 40.64 25.4 90) (unit 1)
-    (in_bom yes) (on_board yes) (fields_autoplaced)
-    (property "Reference" "R14" (id 0) (at 40.64 20.8112 90))
-    (property "Value" "0" (id 1) (at 40.64 23.3481 90))
-    (property "Footprint" "Resistor_SMD:R_0402_1005Metric" (id 2) (at 40.64 25.4 0)
-      (effects (font (size 1.27 1.27)) hide)
-    )
-    (property "Datasheet" "~" (id 3) (at 40.64 25.4 0)
-      (effects (font (size 1.27 1.27)) hide)
-    )
-    (property "MPN" "RC0402JR-070RL" (id 4) (at 40.64 25.4 0)
-      (effects (font (size 1.27 1.27)) hide)
-    )
