File: MotorController/POWER.kicad_sch (KiCad schematic)
At the start: 39 parts, among them U1 LMR12010YMKE, U14 INA280A3IDCKR, U2 INA280A3IDCKR, U3 INA280A3IDCKR, U4 AP7366-W5-7

Commit message: The monstrosity is almost done
The monstrosity is almost done
Connections:
- net +BATT: now also R37.2; no longer R37.1
- net +RMOTOR_VBAT: now also R37.1; no longer R37.2
Other:
- moved on the sheet: R37
Changed lines of the file:
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@@
   (junction (at 212.09 33.02) (diameter 0) (color 0 0 0 0)
   )
+  (junction (at 163.83 129.54) (diameter 0) (color 0 0 0 0)
+  )
   (junction (at 97.79 83.82) (diameter 0) (color 0 0 0 0)
   )
@@
   (junction (at 166.37 139.7) (diameter 0) (color 0 0 0 0)
   )
+  (junction (at 120.65 33.02) (diameter 0) (color 0 0 0 0)
+  )
+  (junction (at 133.35 73.66) (diameter 0) (color 0 0 0 0)
+  )
+  (junction (at 196.85 44.45) (diameter 0) (color 0 0 0 0)
+  )
+  (junction (at 86.36 83.82) (diameter 0) (color 0 0 0 0)
+  )
+  (junction (at 97.79 44.45) (diameter 0) (color 0 0 0 0)
+  )
+  (junction (at 209.55 22.86) (diameter 0) (color 0 0 0 0)
+  )
   (junction (at 176.53 129.54) (diameter 0) (color 0 0 0 0)
   )
-  (junction (at 120.65 33.02) (diameter 0) (color 0 0 0 0)
-  )
-  (junction (at 133.35 73.66) (diameter 0) (color 0 0 0 0)
-  )
-  (junction (at 196.85 44.45) (diameter 0) (color 0 0 0 0)
-  )
-  (junction (at 86.36 83.82) (diameter 0) (color 0 0 0 0)
-  )
-  (junction (at 97.79 44.45) (diameter 0) (color 0 0 0 0)
-  )
-  (junction (at 209.55 22.86) (diameter 0) (color 0 0 0 0)
-  )
   (junction (at 180.34 83.82) (diameter 0) (color 0 0 0 0)
   )
@@
   (junction (at 222.25 22.86) (diameter 0) (color 0 0 0 0)
   )
-  (junction (at 163.83 129.54) (diameter 0) (color 0 0 0 0)
-  )
   (junction (at 123.19 22.86) (diameter 0) (color 0 0 0 0)
   )
@@
     (stroke (width 0) (type default) (color 0 0 0 0))
   )
+  (wire (pts (xy 172.72 129.54) (xy 176.53 129.54))
+    (stroke (width 0) (type default) (color 0 0 0 0))
+  )
   (wire (pts (xy 180.34 83.82) (xy 180.34 87.63))
     (stroke (width 0) (type default) (color 0 0 0 0))
@@
     (stroke (width 0) (type default) (color 0 0 0 0))
   )
+  (wire (pts (xy 163.83 129.54) (xy 167.64 129.54))
+    (stroke (width 0) (type default) (color 0 0 0 0))
+  )
   (wire (pts (xy 256.54 83.82) (xy 262.89 83.82))
     (stroke (width 0) (type default) (color 0 0 0 0))
@@
     (stroke (width 0) (type default) (color 0 0 0 0))
   )
-  (wire (pts (xy 163.83 129.54) (xy 167.64 129.54))
-    (stroke (width 0) (type default) (color 0 0 0 0))
-  )
   (wire (pts (xy 166.37 83.82) (xy 161.29 83.82))
     (stroke (width 0) (type default) (color 0 0 0 0))
@@
   )
   (wire (pts (xy 133.35 73.66) (xy 133.35 76.2))
-    (stroke (width 0) (type default) (color 0 0 0 0))
-  )
-  (wire (pts (xy 172.72 129.54) (xy 176.53 129.54))
     (stroke (width 0) (type default) (color 0 0 0 0))
   )
@@
     (pin "5")
   )
-  (symbol (lib_id "Device:R_Small_US") (at 170.18 129.54 90) (unit 1)
-    (in_bom yes) (on_board yes) (fields_autoplaced)
-    (property "Reference" "R37" (id 0) (at 170.18 124.9512 90))
-    (property "Value" "0.2mOhms" (id 1) (at 170.18 127.4881 90))
+  (symbol (lib_id "Device:R_Small_US") (at 170.18 129.54 270) (unit 1)
+    (in_bom yes) (on_board yes) (fields_autoplaced)
+    (property "Reference" "R37" (id 0) (at 170.18 123.19 90))
+    (property "Value" "0.2mOhms" (id 1) (at 170.18 125.73 90))
     (property "Footprint" "Footprints:RES_WSK12161L000FEA" (id 2) (at 170.18 129.54 0)
       (effects (font (size 1.27 1.27)) hide)
