File: MotorController/RMOTOR.kicad_sch (KiCad schematic)
At the start: 0 parts

Commit message: Updates
Updates
Parts:
- added C? (x2): 40nF, symbol Device:C_Small
- added C? (x2): 1uF, symbol Device:C_Small
- added D? (x4): D_Small_Filled, symbol Device:D_Small_Filled
- added M?: Motor_DC, symbol Motor:Motor_DC
- added Q? (x4): Q_NMOS_GDS, symbol Device:Q_NMOS_GDS
- added R? (x2): DNU, symbol Device:R_Small_US
- added R?: 0, symbol Device:R_Small_US
- added U? (x2): 2EDL8024GX, symbol ProjectSymbols:2EDL8024GX
Connections:
- new net: C?.2, D?.1 (K), D?.2 (A), M?.2 (-), Q?.2 (D), Q?.3 (S), U?.4 (HS)
- new net: C?.2, D?.1 (K), D?.2 (A), M?.1 (+), Q?.2 (D), Q?.3 (S), U?.4 (HS)
- new net: Q?.1 (G), U?.8 (LO) (x2)
- new net: Q?.1 (G), U?.3 (HO) (x2)
- new net +3V3: R?.1
- new net +5V: R?.1
- new net +BATT: D?.1 (K), D?.1 (K), Q?.2 (D), Q?.2 (D), R?.1
- new net +VDD: C?.1, C?.1, R?.2, R?.2, R?.2, U?.1 (VDD), U?.1 (VDD)
- new net GND: C?.2, C?.2, D?.2 (A), D?.2 (A), Q?.3 (S), Q?.3 (S), U?.7 (VSS), U?.7 (VSS), U?.9 (VSS), U?.9 (VSS)
- new net LBOOTSTRAP: C?.1, U?.2 (HB)
- new net RBOOTSTRAP: C?.1, U?.2 (HB)
- new net RMOTOR_BACKWARDS: U?.5 (HI), U?.6 (LI)
- new net RMOTOR_FORWARD: U?.5 (HI), U?.6 (LI)

Commit message: More updates
Parts:
- removed C? (x2): 40nF, symbol Device:C_Small
- removed C? (x2): 1uF, symbol Device:C_Small
- removed D? (x4): D_Small_Filled, symbol Device:D_Small_Filled
- removed M?: Motor_DC, symbol Motor:Motor_DC
- removed Q? (x4): Q_NMOS_GDS, symbol Device:Q_NMOS_GDS
- removed R? (x2): DNU, symbol Device:R_Small_US
- removed R?: 0, symbol Device:R_Small_US
- removed U? (x2): 2EDL8024GX, symbol ProjectSymbols:2EDL8024GX
- added C? (x2): 40nF, symbol Device:C_Small
- added C? (x2): 1uF, symbol Device:C_Small
- added C?: 1000uF, symbol Device:C_Small
- added D? (x8): D_Small_Filled, symbol Device:D_Small_Filled
- added M?: Motor_DC, symbol Motor:Motor_DC
- added Q? (x4): Q_NMOS_GDS, symbol Device:Q_NMOS_GDS
- added R? (x4): 2, symbol Device:R_Small_US
- added R? (x2): DNU, symbol Device:R_Small_US
- added R?: 0, symbol Device:R_Small_US
- added U? (x2): 2EDL8024GX, symbol ProjectSymbols:2EDL8024GX
Connections:
- net +3V3: now also R?.1
- net +5V: now also R?.1
- net +BATT: now also C?.1, D?.1 (K), D?.1 (K), Q?.2 (D), Q?.2 (D), R?.1
- net +VDD: now also C?.1, C?.1, R?.2, R?.2, R?.2, U?.1 (VDD), U?.1 (VDD)
- net GND: now also C?.2, C?.2, C?.2, D?.2 (A), D?.2 (A), Q?.3 (S), Q?.3 (S), U?.7 (VSS), U?.7 (VSS), U?.9 (VSS), U?.9 (VSS)
- net LBOOTSTRAP: now also C?.1, U?.2 (HB)
- net RBOOTSTRAP: now also C?.1, U?.2 (HB)
- net RMOTOR_BACKWARDS: now also U?.5 (HI), U?.6 (LI)
- net RMOTOR_FORWARD: now also U?.5 (HI), U?.6 (LI)
- new net: C?.2, D?.1 (K), D?.2 (A), M?.1 (+), Q?.2 (D), Q?.3 (S), U?.4 (HS)
- new net: D?.2 (A), Q?.1 (G), R?.1 (x2)
- new net: D?.1 (K), R?.2, U?.3 (HO) (x2)
- new net: D?.2 (A), Q?.1 (G), R?.2 (x2)
- new net: C?.2, D?.1 (K), D?.2 (A), M?.2 (-), Q?.2 (D), Q?.3 (S), U?.4 (HS)
- new net: D?.1 (K), R?.1, U?.8 (LO) (x2)

Commit message: Updates
Parts:
- C20, C24: renamed from C?; footprint (none) -> Capacitor_SMD:C_0603_1608Metric; MPN (none) -> CC0603KRX5R8BB105
- C21, C23: renamed from C?; footprint (none) -> Capacitor_SMD:C_0603_1608Metric; MPN (none) -> CC0603KRX7R8BB393
- C22: renamed from C?; value 1000uF -> 330uF; footprint (none) -> Capacitor_SMD:CP_Elec_10x10; MPN (none) -> A771MS337M1VLAS014
- D12, D13, D14, D15, D16, D17, D18, D19: renamed from D?; MPN (none) -> S1A-13-F
- M2: renamed from M?; footprint (none) -> Connector_PinHeader_2.54mm:PinHeader_1x02_P2.54mm_Vertical
- Q5, Q6, Q7, Q8: renamed from Q?; footprint (none) -> Footprints:TRANS_SSM6K513NU-LF; MPN (none) -> FDD8447L
- R21, R22, R23: renamed from R?; footprint (none) -> Resistor_SMD:R_0603_1608Metric; MPN (none) -> RC0603FR-070RL
- R24, R25, R26, R27: renamed from R?; footprint (none) -> Resistor_SMD:R_0603_1608Metric; MPN (none) -> RC0603FR-072RL
- U11, U12: renamed from U?; footprint (none) -> Package_DFN_QFN:DFN-8-1EP_4x4mm_P0.8mm_EP2.3x3.24mm; MPN (none) -> 2EDL8024GX

Commit message: Changes
Changes
Parts:
- removed D12, D13, D18, D19: D_Small_Filled, symbol Device:D_Small_Filled
- removed Q5, Q6, Q7, Q8: Q_NMOS_GDS, Footprints:TRANS_SSM6K513NU-LF, symbol Device:Q_NMOS_GDS
- added D? (x4): D_Small_Filled, Diode_SMD:D_SOD-323, symbol Device:D_Small_Filled
- added Q5, Q6, Q7, Q8: SSM6K513NU-LF, Footprints:TRANS_SSM6K513NU-LF, symbol ProjectSymbols:SSM6K513NU-LF
- D14, D15, D16, D17: MPN S1A-13-F -> (none)
Connections:
- net +BATT: now also Q5.1, Q5.2, Q5.5, Q5.6, Q5.7, Q7.1, Q7.2, Q7.5, Q7.6, Q7.7
- net GND: now also Q6.4, Q6.8, Q8.4, Q8.8
- net at C21.2, D14.2 (A), D15.1 (K)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: now also Q5.4, Q5.8, Q6.1, Q6.2, Q6.5, Q6.6, Q6.7
- net at R24.1: now also D?.2 (A), Q5.3
- net at R26.1: now also D?.2 (A), Q7.3
- net at R26.2, U12.3 (HO): now also D?.1 (K)
- net at R24.2, U11.3 (HO): now also D?.1 (K)
- net at R27.2: now also D?.2 (A), Q8.3
- net at C23.2, D16.2 (A), D17.1 (K)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: now also Q7.4, Q7.8, Q8.1, Q8.2, Q8.5, Q8.6, Q8.7
- net at R25.1, U11.8 (LO): now also D?.1 (K)
- net at R25.2: now also D?.2 (A), Q6.3
- net at R27.1, U12.8 (LO): now also D?.1 (K)

Commit message: So many updates
Parts:
- removed D14, D16: D_Small_Filled, symbol Device:D_Small_Filled
- added D18, D19: D_Small_Filled, Footprints:TO-277B, symbol Device:D_Small_Filled
- C20, C24: footprint Capacitor_SMD:C_0603_1608Metric -> Capacitor_SMD:C_0402_1005Metric; MPN CC0603KRX5R8BB105 -> CC0402KRX5R8BB105
- C21, C23: value 40nF -> 33nF; footprint Capacitor_SMD:C_0603_1608Metric -> Capacitor_SMD:C_0402_1005Metric; MPN CC0603KRX7R8BB393 -> CC0402KRX7R9BB333
- C22: footprint Capacitor_SMD:CP_Elec_10x10 -> Connector_PinHeader_2.54mm:PinHeader_1x02_P2.54mm_Vertical; MPN A771MS337M1VLAS014 -> (none)
- D15, D17: footprint (none) -> Footprints:TO-277B; MPN (none) -> MBR1560S
- R21: footprint Resistor_SMD:R_0603_1608Metric -> Resistor_SMD:R_0402_1005Metric; MPN RC0603FR-070RL -> RC0402JR-070RL
- R22, R23: footprint Resistor_SMD:R_0603_1608Metric -> Resistor_SMD:R_0402_1005Metric; MPN RC0603FR-070RL -> RC0402JR-0710KL
- R24, R25, R26, R27: footprint Resistor_SMD:R_0603_1608Metric -> Resistor_SMD:R_0402_1005Metric; MPN RC0603FR-072RL -> RC0402FR-072RL
- gave numbers to parts that had none: 4
Connections:
- net +BATT: now also D17.1 (K), D18.1 (K)
- net GND: now also D19.2 (A); no longer D17.2 (A)
- net at C23.2, M2.2 (-), Q7.4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: now also D18.2 (A), D19.1 (K); no longer D17.1 (K)
- net at C21.2, D15.1 (K), M2.1 (+)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: now also D17.2 (A)

Commit message: my god
my god
Connections:
- net +VDD renamed +VDD_R
- net LBOOTSTRAP renamed RLBOOTSTRAP
- net RBOOTSTRAP renamed RRBOOTSTRAP
Changed lines of the file:
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@@
     (stroke (width 0) (type default) (color 0 0 0 0))
   )
-  (global_label "+VDD" (shape input) (at 43.18 88.9 180) (fields_autoplaced)
+  (global_label "+VDD_R" (shape input) (at 269.24 93.98 0) (fields_autoplaced)
+    (effects (font (size 1.27 1.27)) (justify left))
+    (property "Intersheet References" "${INTERSHEET_REFS}" (id 0) (at 279.0917 94.0594 0)
+      (effects (font (size 1.27 1.27)) (justify left) hide)
+    )
+  )
+  (global_label "RRBOOTSTRAP" (shape bidirectional) (at 229.87 111.76 0) (fields_autoplaced)
+    (effects (font (size 1.27 1.27)) (justify left))
+    (property "Intersheet References" "${INTERSHEET_REFS}" (id 0) (at 245.5274 111.6806 0)
+      (effects (font (size 1.27 1.27)) (justify left) hide)
+    )
+  )
+  (global_label "RLBOOTSTRAP" (shape bidirectional) (at 78.74 106.68 180) (fields_autoplaced)
     (effects (font (size 1.27 1.27)) (justify right))
-    (property "Intersheet References" "${INTERSHEET_REFS}" (id 0) (at 35.5659 88.9794 0)
+    (property "Intersheet References" "${INTERSHEET_REFS}" (id 0) (at 63.3245 106.6006 0)
       (effects (font (size 1.27 1.27)) (justify right) hide)
     )
   )
-  (global_label "RBOOTSTRAP" (shape bidirectional) (at 229.87 111.76 0) (fields_autoplaced)
+  (global_label "+VDD_R" (shape output) (at 48.26 74.93 0) (fields_autoplaced)
     (effects (font (size 1.27 1.27)) (justify left))
-    (property "Intersheet References" "${INTERSHEET_REFS}" (id 0) (at 244.2574 111.6806 0)
+    (property "Intersheet References" "${INTERSHEET_REFS}" (id 0) (at 58.1117 74.8506 0)
       (effects (font (size 1.27 1.27)) (justify left) hide)
     )
   )
-  (global_label "LBOOTSTRAP" (shape bidirectional) (at 78.74 106.68 180) (fields_autoplaced)
+  (global_label "+VDD_R" (shape input) (at 43.18 88.9 180) (fields_autoplaced)
     (effects (font (size 1.27 1.27)) (justify right))
-    (property "Intersheet References" "${INTERSHEET_REFS}" (id 0) (at 64.5945 106.6006 0)
+    (property "Intersheet References" "${INTERSHEET_REFS}" (id 0) (at 33.3283 88.9794 0)
       (effects (font (size 1.27 1.27)) (justify right) hide)
     )
   )
-  (global_label "+VDD" (shape output) (at 48.26 74.93 0) (fields_autoplaced)
-    (effects (font (size 1.27 1.27)) (justify left))
-    (property "Intersheet References" "${INTERSHEET_REFS}" (id 0) (at 55.8741 74.8506 0)
-      (effects (font (size 1.27 1.27)) (justify left) hide)
-    )
-  )
-  (global_label "LBOOTSTRAP" (shape bidirectional) (at 107.95 77.47 180) (fields_autoplaced)
+  (global_label "RLBOOTSTRAP" (shape bidirectional) (at 107.95 77.47 180) (fields_autoplaced)
     (effects (font (size 1.27 1.27)) (justify right))
-    (property "Intersheet References" "${INTERSHEET_REFS}" (id 0) (at 93.8045 77.3906 0)
+    (property "Intersheet References" "${INTERSHEET_REFS}" (id 0) (at 92.5345 77.3906 0)
       (effects (font (size 1.27 1.27)) (justify right) hide)
     )
   )
-  (global_label "+VDD" (shape input) (at 269.24 93.98 0) (fields_autoplaced)
+  (global_label "RRBOOTSTRAP" (shape bidirectional) (at 203.2 77.47 0) (fields_autoplaced)
     (effects (font (size 1.27 1.27)) (justify left))
-    (property "Intersheet References" "${INTERSHEET_REFS}" (id 0) (at 276.8541 94.0594 0)
+    (property "Intersheet References" "${INTERSHEET_REFS}" (id 0) (at 218.8574 77.3906 0)
       (effects (font (size 1.27 1.27)) (justify left) hide)
     )
-  )
-  (global_label "RBOOTSTRAP" (shape bidirectional) (at 203.2 77.47 0) (fields_autoplaced)
-    (effects (font (size 1.27 1.27)) (justify left))
-    (property "Intersheet References" "${INTERSHEET_REFS}" (id 0) (at 217.5874 77.3906 0)
-      (effects (font (size 1.27 1.27)) (justify left) hide)
-    )

Commit message: The monstrosity is almost done
The monstrosity is almost done
Parts:
- removed R21: 0, Resistor_SMD:R_0402_1005Metric, symbol Device:R_Small_US
Changed lines of the file:
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@@
-    (stroke (width 0) (type default) (color 0 0 0 0))
-  )
-  (wire (pts (xy 34.29 67.31) (xy 38.1 67.31))
     (stroke (width 0) (type default) (color 0 0 0 0))
   )
@@
     (stroke (width 0) (type default) (color 0 0 0 0))
   )
-  (wire (pts (xy 45.72 67.31) (xy 45.72 74.93))
-    (stroke (width 0) (type default) (color 0 0 0 0))
-  )
   (wire (pts (xy 127 67.31) (xy 121.92 67.31))
     (stroke (width 0) (type default) (color 0 0 0 0))
@@
   )
   (wire (pts (xy 184.15 78.74) (xy 184.15 82.55))
-    (stroke (width 0) (type default) (color 0 0 0 0))
-  )
-  (wire (pts (xy 43.18 67.31) (xy 45.72 67.31))
     (stroke (width 0) (type default) (color 0 0 0 0))
   )
@@
   )
   (hierarchical_label "+5V" (shape input) (at 34.29 74.93 180)
-    (effects (font (size 1.27 1.27)) (justify right))
-  )
-  (hierarchical_label "+3V3" (shape input) (at 34.29 67.31 180)
     (effects (font (size 1.27 1.27)) (justify right))
   )
@@
     (pin "1")
   )
-  (symbol (lib_id "Device:R_Small_US") (at 40.64 67.31 90) (unit 1)
-    (in_bom yes) (on_board yes) (fields_autoplaced)
-    (property "Reference" "R21" (id 0) (at 40.64 62.7212 90))
-    (property "Value" "0" (id 1) (at 40.64 65.2581 90))
-    (property "Footprint" "Resistor_SMD:R_0402_1005Metric" (id 2) (at 40.64 67.31 0)
-      (effects (font (size 1.27 1.27)) hide)
-    )
-    (property "Datasheet" "~" (id 3) (at 40.64 67.31 0)
-      (effects (font (size 1.27 1.27)) hide)
-    )
-    (property "MPN" "RC0402JR-070RL" (id 4) (at 40.64 67.31 0)
-      (effects (font (size 1.27 1.27)) hide)
-    )
-    (pin "1")
-    (pin "2")
-  )
   (symbol (lib_id "Device:D_Small_Filled") (at 185.42 114.3 270) (unit 1)
