File: MotorController/FLASH.kicad_sch (KiCad schematic)
At the start: 0 parts

Commit message: Schematic Updates
Parts:
- added C?: C_Small, symbol Device:C_Small
- added R? (x2): 0, symbol Device:R_Small_US
- added U?: MT25QL128ABA1, symbol ProjectSymbols:MT25QL128ABA1
Connections:
- new net: R?.2, U?.7 (DQ3/~{HOLD})
- new net: R?.1, U?.3 (~{W}/DQ2)
- new net +3V3: C?.1, U?.8 (VCC)
- new net FLASH_MISO: U?.2 (DQ1/MISO)
- new net FLASH_MOSI: U?.5 (DQ0/MOSI)
- new net FLASH_SCK: U?.6 (CLK)
- new net GND: C?.2, U?.4 (VSS)
- new net ~{FLASH_CS}: U?.1 (~{CS})
- new net ~{FLASH_HOLD}: R?.1
- new net ~{FLASH_W}: R?.2
Changed lines of the file:
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@@
 (kicad_sch (version 20211123) (generator eeschema)
   (paper "A4")
+  (junction (at 107.95 67.31) (diameter 0) (color 0 0 0 0)
+  )
+  (wire (pts (xy 158.75 67.31) (xy 163.83 67.31))
+    (stroke (width 0) (type default) (color 0 0 0 0))
+  )
+  (wire (pts (xy 184.15 77.47) (xy 189.23 77.47))
+    (stroke (width 0) (type default) (color 0 0 0 0))
+  )
+  (wire (pts (xy 184.15 74.93) (xy 189.23 74.93))
+    (stroke (width 0) (type default) (color 0 0 0 0))
+  )
+  (wire (pts (xy 107.95 74.93) (xy 107.95 77.47))
+    (stroke (width 0) (type default) (color 0 0 0 0))
+  )
+  (wire (pts (xy 158.75 69.85) (xy 163.83 69.85))
+    (stroke (width 0) (type default) (color 0 0 0 0))
+  )
+  (wire (pts (xy 161.29 83.82) (xy 161.29 81.28))
+    (stroke (width 0) (type default) (color 0 0 0 0))
+  )
+  (wire (pts (xy 132.08 72.39) (xy 134.62 72.39))
+    (stroke (width 0) (type default) (color 0 0 0 0))
+  )
+  (wire (pts (xy 104.14 67.31) (xy 107.95 67.31))
+    (stroke (width 0) (type default) (color 0 0 0 0))
+  )
+  (wire (pts (xy 107.95 67.31) (xy 134.62 67.31))
+    (stroke (width 0) (type default) (color 0 0 0 0))
+  )
+  (wire (pts (xy 107.95 69.85) (xy 107.95 67.31))
+    (stroke (width 0) (type default) (color 0 0 0 0))
+  )
+  (wire (pts (xy 158.75 74.93) (xy 179.07 74.93))
+    (stroke (width 0) (type default) (color 0 0 0 0))
+  )
+  (wire (pts (xy 161.29 81.28) (xy 158.75 81.28))
+    (stroke (width 0) (type default) (color 0 0 0 0))
+  )
+  (wire (pts (xy 132.08 81.28) (xy 134.62 81.28))
+    (stroke (width 0) (type default) (color 0 0 0 0))
+  )
+  (wire (pts (xy 158.75 77.47) (xy 179.07 77.47))
+    (stroke (width 0) (type default) (color 0 0 0 0))
+  )
+  (hierarchical_label "FLASH_MISO" (shape output) (at 163.83 69.85 0)
+    (effects (font (size 1.27 1.27)) (justify left))
+  )
+  (hierarchical_label "FLASH_MOSI" (shape input) (at 163.83 67.31 0)
+    (effects (font (size 1.27 1.27)) (justify left))
+  )
+  (hierarchical_label "~{FLASH_HOLD}" (shape input) (at 189.23 77.47 0)
+    (effects (font (size 1.27 1.27)) (justify left))
+  )
+  (hierarchical_label "~{FLASH_W}" (shape input) (at 189.23 74.93 0)
+    (effects (font (size 1.27 1.27)) (justify left))
+  )
+  (hierarchical_label "+3V3" (shape input) (at 104.14 67.31 180)
+    (effects (font (size 1.27 1.27)) (justify right))
+  )
+  (hierarchical_label "FLASH_SCK" (shape input) (at 132.08 81.28 180)
+    (effects (font (size 1.27 1.27)) (justify right))
+  )
+  (hierarchical_label "~{FLASH_CS}" (shape input) (at 132.08 72.39 180)
+    (effects (font (size 1.27 1.27)) (justify right))
+  )
+  (symbol (lib_id "Device:C_Small") (at 107.95 72.39 0) (unit 1)
+    (in_bom yes) (on_board yes) (fields_autoplaced)
+    (property "Reference" "C?" (id 0) (at 110.49 71.1262 0)
+      (effects (font (size 1.27 1.27)) (justify left))
+    )
+    (property "Value" "C_Small" (id 1) (at 110.49 73.6662 0)
+      (effects (font (size 1.27 1.27)) (justify left))
+    )
+    (property "Footprint" "" (id 2) (at 107.95 72.39 0)
+      (effects (font (size 1.27 1.27)) hide)
+    )
+    (property "Datasheet" "~" (id 3) (at 107.95 72.39 0)
+      (effects (font (size 1.27 1.27)) hide)
+    )
+    (pin "1")
+    (pin "2")
+  )
+  (symbol (lib_id "power:GND") (at 161.29 83.82 0) (unit 1)
+    (in_bom yes) (on_board yes) (fields_autoplaced)
+    (property "Reference" "#PWR?" (id 0) (at 161.29 90.17 0)
+      (effects (font (size 1.27 1.27)) hide)
+    )
+    (property "Value" "GND" (id 1) (at 161.29 88.9 0)
+      (effects (font (size 1.27 1.27)) hide)
+    )
+    (property "Footprint" "" (id 2) (at 161.29 83.82 0)
+      (effects (font (size 1.27 1.27)) hide)
+    )
+    (property "Datasheet" "" (id 3) (at 161.29 83.82 0)
+      (effects (font (size 1.27 1.27)) hide)
+    )
+    (pin "1")
+  )
+  (symbol (lib_id "Device:R_Small_US") (at 181.61 77.47 270) (unit 1)
+    (in_bom yes) (on_board yes)
+    (property "Reference" "R?" (id 0) (at 181.61 82.55 90))
+    (property "Value" "0" (id 1) (at 181.61 80.01 90))
+    (property "Footprint" "" (id 2) (at 181.61 77.47 0)
+      (effects (font (size 1.27 1.27)) hide)
+    )
+    (property "Datasheet" "~" (id 3) (at 181.61 77.47 0)
+      (effects (font (size 1.27 1.27)) hide)
+    )
+    (pin "1")
+    (pin "2")
+  )
+  (symbol (lib_id "power:GND") (at 107.95 77.47 0) (unit 1)
+    (in_bom yes) (on_board yes) (fields_autoplaced)
+    (property "Reference" "#PWR?" (id 0) (at 107.95 83.82 0)
+      (effects (font (size 1.27 1.27)) hide)
+    )
+    (property "Value" "GND" (id 1) (at 107.95 82.55 0)
+      (effects (font (size 1.27 1.27)) hide)
+    )
+    (property "Footprint" "" (id 2) (at 107.95 77.47 0)
+      (effects (font (size 1.27 1.27)) hide)
+    )
+    (property "Datasheet" "" (id 3) (at 107.95 77.47 0)
+      (effects (font (size 1.27 1.27)) hide)
+    )
+    (pin "1")
+  )
+  (symbol (lib_id "Device:R_Small_US") (at 181.61 74.93 90) (unit 1)
+    (in_bom yes) (on_board yes) (fields_autoplaced)
+    (property "Reference" "R?" (id 0) (at 181.61 68.58 90))
+    (property "Value" "0" (id 1) (at 181.61 71.12 90))
+    (property "Footprint" "" (id 2) (at 181.61 74.93 0)
+      (effects (font (size 1.27 1.27)) hide)
+    )
+    (property "Datasheet" "~" (id 3) (at 181.61 74.93 0)
+      (effects (font (size 1.27 1.27)) hide)
+    )
+    (pin "1")
+    (pin "2")
+  )
+  (symbol (lib_id "ProjectSymbols:MT25QL128ABA1") (at 144.78 71.12 0) (unit 1)
+    (in_bom yes) (on_board yes) (fields_autoplaced)
+    (property "Reference" "U?" (id 0) (at 146.685 60.96 0))
+    (property "Value" "MT25QL128ABA1" (id 1) (at 146.685 63.5 0))
+    (property "Footprint" "" (id 2) (at 144.78 55.88 0)
+      (effects (font (size 1.27 1.27)) hide)
+    )
+    (property "Datasheet" "" (id 3) (at 144.78 55.88 0)
+      (effects (font (size 1.27 1.27)) hide)
+    )
+    (pin "1")
+    (pin "2")
+    (pin "3")
+    (pin "4")
+    (pin "5")
+    (pin "6")
+    (pin "7")
+    (pin "8")
+  )
 )

Commit message: Updates
Parts:
- C25: renamed from C?; value C_Small -> 0.1uF; footprint (none) -> Capacitor_SMD:C_0603_1608Metric; MPN (none) -> CC0603JRX7R8BB104
- R32, R33: renamed from R?; footprint (none) -> Resistor_SMD:R_0603_1608Metric; MPN (none) -> RC0603FR-070RL
- U13: renamed from U?; footprint (none) -> Footprints:SOIC127P780X200-8N; MPN (none) -> MT25QL128ABA1
Changed lines of the file:
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@@
   (symbol (lib_id "Device:C_Small") (at 107.95 72.39 0) (unit 1)
     (in_bom yes) (on_board yes) (fields_autoplaced)
-    (property "Reference" "C?" (id 0) (at 110.49 71.1262 0)
+    (property "Reference" "C25" (id 0) (at 110.49 71.1262 0)
       (effects (font (size 1.27 1.27)) (justify left))
     )
-    (property "Value" "C_Small" (id 1) (at 110.49 73.6662 0)
+    (property "Value" "0.1uF" (id 1) (at 110.49 73.6662 0)
       (effects (font (size 1.27 1.27)) (justify left))
     )
-    (property "Footprint" "" (id 2) (at 107.95 72.39 0)
+    (property "Footprint" "Capacitor_SMD:C_0603_1608Metric" (id 2) (at 107.95 72.39 0)
       (effects (font (size 1.27 1.27)) hide)
     )
     (property "Datasheet" "~" (id 3) (at 107.95 72.39 0)
+      (effects (font (size 1.27 1.27)) hide)
+    )
+    (property "MPN" "CC0603JRX7R8BB104" (id 4) (at 107.95 72.39 0)
       (effects (font (size 1.27 1.27)) hide)
     )
@@
   (symbol (lib_id "power:GND") (at 161.29 83.82 0) (unit 1)
     (in_bom yes) (on_board yes) (fields_autoplaced)
-    (property "Reference" "#PWR?" (id 0) (at 161.29 90.17 0)
+    (property "Reference" "#PWR046" (id 0) (at 161.29 90.17 0)
       (effects (font (size 1.27 1.27)) hide)
     )
@@
   (symbol (lib_id "Device:R_Small_US") (at 181.61 77.47 270) (unit 1)
     (in_bom yes) (on_board yes)
-    (property "Reference" "R?" (id 0) (at 181.61 82.55 90))
+    (property "Reference" "R33" (id 0) (at 181.61 82.55 90))
     (property "Value" "0" (id 1) (at 181.61 80.01 90))
-    (property "Footprint" "" (id 2) (at 181.61 77.47 0)
+    (property "Footprint" "Resistor_SMD:R_0603_1608Metric" (id 2) (at 181.61 77.47 0)
       (effects (font (size 1.27 1.27)) hide)
     )
     (property "Datasheet" "~" (id 3) (at 181.61 77.47 0)
+      (effects (font (size 1.27 1.27)) hide)
+    )
+    (property "MPN" "RC0603FR-070RL" (id 4) (at 181.61 77.47 0)
       (effects (font (size 1.27 1.27)) hide)
     )
@@
   (symbol (lib_id "power:GND") (at 107.95 77.47 0) (unit 1)
     (in_bom yes) (on_board yes) (fields_autoplaced)
-    (property "Reference" "#PWR?" (id 0) (at 107.95 83.82 0)
+    (property "Reference" "#PWR045" (id 0) (at 107.95 83.82 0)
       (effects (font (size 1.27 1.27)) hide)
     )
@@
   (symbol (lib_id "Device:R_Small_US") (at 181.61 74.93 90) (unit 1)
     (in_bom yes) (on_board yes) (fields_autoplaced)
-    (property "Reference" "R?" (id 0) (at 181.61 68.58 90))
+    (property "Reference" "R32" (id 0) (at 181.61 68.58 90))
     (property "Value" "0" (id 1) (at 181.61 71.12 90))
-    (property "Footprint" "" (id 2) (at 181.61 74.93 0)
+    (property "Footprint" "Resistor_SMD:R_0603_1608Metric" (id 2) (at 181.61 74.93 0)
       (effects (font (size 1.27 1.27)) hide)
     )
     (property "Datasheet" "~" (id 3) (at 181.61 74.93 0)
+      (effects (font (size 1.27 1.27)) hide)
+    )
+    (property "MPN" "RC0603FR-070RL" (id 4) (at 181.61 74.93 0)
       (effects (font (size 1.27 1.27)) hide)
     )
@@
   (symbol (lib_id "ProjectSymbols:MT25QL128ABA1") (at 144.78 71.12 0) (unit 1)
     (in_bom yes) (on_board yes) (fields_autoplaced)
-    (property "Reference" "U?" (id 0) (at 146.685 60.96 0))
+    (property "Reference" "U13" (id 0) (at 146.685 60.96 0))
     (property "Value" "MT25QL128ABA1" (id 1) (at 146.685 63.5 0))
-    (property "Footprint" "" (id 2) (at 144.78 55.88 0)
+    (property "Footprint" "Footprints:SOIC127P780X200-8N" (id 2) (at 144.78 55.88 0)
       (effects (font (size 1.27 1.27)) hide)
     )
@@
       (effects (font (size 1.27 1.27)) hide)
     )
+    (property "MPN" "MT25QL128ABA1" (id 4) (at 144.78 71.12 0)
+      (effects (font (size 1.27 1.27)) hide)
+    )

Commit message: So many updates
Parts:
- C25: footprint Capacitor_SMD:C_0603_1608Metric -> Capacitor_SMD:C_0402_1005Metric; MPN CC0603JRX7R8BB104 -> CC0402KPX7R8BB104
- R32, R33: footprint Resistor_SMD:R_0603_1608Metric -> Resistor_SMD:R_0402_1005Metric; MPN RC0603FR-070RL -> RC0402JR-070RL
Changed lines of the file:
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@@
       (effects (font (size 1.27 1.27)) (justify left))
     )
-    (property "Footprint" "Capacitor_SMD:C_0603_1608Metric" (id 2) (at 107.95 72.39 0)
+    (property "Footprint" "Capacitor_SMD:C_0402_1005Metric" (id 2) (at 107.95 72.39 0)
       (effects (font (size 1.27 1.27)) hide)
     )
@@
       (effects (font (size 1.27 1.27)) hide)
     )
-    (property "MPN" "CC0603JRX7R8BB104" (id 4) (at 107.95 72.39 0)
+    (property "MPN" "CC0402KPX7R8BB104" (id 4) (at 107.95 72.39 0)
       (effects (font (size 1.27 1.27)) hide)
     )
@@
     (property "Reference" "R33" (id 0) (at 181.61 82.55 90))
     (property "Value" "0" (id 1) (at 181.61 80.01 90))
-    (property "Footprint" "Resistor_SMD:R_0603_1608Metric" (id 2) (at 181.61 77.47 0)
+    (property "Footprint" "Resistor_SMD:R_0402_1005Metric" (id 2) (at 181.61 77.47 0)
       (effects (font (size 1.27 1.27)) hide)
     )
@@
       (effects (font (size 1.27 1.27)) hide)
     )
-    (property "MPN" "RC0603FR-070RL" (id 4) (at 181.61 77.47 0)
+    (property "MPN" "RC0402JR-070RL" (id 4) (at 181.61 77.47 0)
       (effects (font (size 1.27 1.27)) hide)
     )
@@
     (property "Reference" "R32" (id 0) (at 181.61 68.58 90))
     (property "Value" "0" (id 1) (at 181.61 71.12 90))
-    (property "Footprint" "Resistor_SMD:R_0603_1608Metric" (id 2) (at 181.61 74.93 0)
+    (property "Footprint" "Resistor_SMD:R_0402_1005Metric" (id 2) (at 181.61 74.93 0)
       (effects (font (size 1.27 1.27)) hide)
     )
@@
       (effects (font (size 1.27 1.27)) hide)
     )
-    (property "MPN" "RC0603FR-070RL" (id 4) (at 181.61 74.93 0)
+    (property "MPN" "RC0402JR-070RL" (id 4) (at 181.61 74.93 0)
       (effects (font (size 1.27 1.27)) hide)
     )

Commit message: ahhhhh
Parts:
- removed R32, R33: 0, Resistor_SMD:R_0402_1005Metric, symbol Device:R_Small_US
Connections:
- no-connect marks 0 -> 2
Changed lines of the file:
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@@
   (junction (at 107.95 67.31) (diameter 0) (color 0 0 0 0)
   )
+  (no_connect (at 158.75 74.93))
+  (no_connect (at 158.75 77.47))
   (wire (pts (xy 158.75 67.31) (xy 163.83 67.31))
-    (stroke (width 0) (type default) (color 0 0 0 0))
-  )
-  (wire (pts (xy 184.15 77.47) (xy 189.23 77.47))
-    (stroke (width 0) (type default) (color 0 0 0 0))
-  )
-  (wire (pts (xy 184.15 74.93) (xy 189.23 74.93))
     (stroke (width 0) (type default) (color 0 0 0 0))
   )
@@
     (stroke (width 0) (type default) (color 0 0 0 0))
   )
-  (wire (pts (xy 158.75 74.93) (xy 179.07 74.93))
-    (stroke (width 0) (type default) (color 0 0 0 0))
-  )
   (wire (pts (xy 161.29 81.28) (xy 158.75 81.28))
     (stroke (width 0) (type default) (color 0 0 0 0))
@@
     (stroke (width 0) (type default) (color 0 0 0 0))
   )
-  (wire (pts (xy 158.75 77.47) (xy 179.07 77.47))
-    (stroke (width 0) (type default) (color 0 0 0 0))
-  )
   (hierarchical_label "FLASH_MISO" (shape output) (at 163.83 69.85 0)
     (effects (font (size 1.27 1.27)) (justify left))
   )
   (hierarchical_label "FLASH_MOSI" (shape input) (at 163.83 67.31 0)
-    (effects (font (size 1.27 1.27)) (justify left))
-  )
-  (hierarchical_label "~{FLASH_HOLD}" (shape input) (at 189.23 77.47 0)
-    (effects (font (size 1.27 1.27)) (justify left))
-  )
-  (hierarchical_label "~{FLASH_W}" (shape input) (at 189.23 74.93 0)
     (effects (font (size 1.27 1.27)) (justify left))
   )
@@
     (pin "1")
   )
-  (symbol (lib_id "Device:R_Small_US") (at 181.61 77.47 270) (unit 1)
-    (in_bom yes) (on_board yes)
-    (property "Reference" "R33" (id 0) (at 181.61 82.55 90))
-    (property "Value" "0" (id 1) (at 181.61 80.01 90))
-    (property "Footprint" "Resistor_SMD:R_0402_1005Metric" (id 2) (at 181.61 77.47 0)
-      (effects (font (size 1.27 1.27)) hide)
-    )
-    (property "Datasheet" "~" (id 3) (at 181.61 77.47 0)
-      (effects (font (size 1.27 1.27)) hide)
-    )
-    (property "MPN" "RC0402JR-070RL" (id 4) (at 181.61 77.47 0)
-      (effects (font (size 1.27 1.27)) hide)
-    )
-    (pin "1")
-    (pin "2")
-  )
   (symbol (lib_id "power:GND") (at 107.95 77.47 0) (unit 1)
     (in_bom yes) (on_board yes) (fields_autoplaced)
@@
     (pin "1")
   )
-  (symbol (lib_id "Device:R_Small_US") (at 181.61 74.93 90) (unit 1)
-    (in_bom yes) (on_board yes) (fields_autoplaced)
-    (property "Reference" "R32" (id 0) (at 181.61 68.58 90))
-    (property "Value" "0" (id 1) (at 181.61 71.12 90))
-    (property "Footprint" "Resistor_SMD:R_0402_1005Metric" (id 2) (at 181.61 74.93 0)
-      (effects (font (size 1.27 1.27)) hide)
-    )
-    (property "Datasheet" "~" (id 3) (at 181.61 74.93 0)
-      (effects (font (size 1.27 1.27)) hide)
-    )
-    (property "MPN" "RC0402JR-070RL" (id 4) (at 181.61 74.93 0)
-      (effects (font (size 1.27 1.27)) hide)
-    )
-    (pin "1")
-    (pin "2")
-  )
   (symbol (lib_id "ProjectSymbols:MT25QL128ABA1") (at 144.78 71.12 0) (unit 1)
