File: MotorController/MCU.kicad_sch (KiCad schematic)
At the start: 0 parts

Commit message: Schematic Updates
Parts:
- added C?: 1uF, symbol Device:C_Small
- added U?: STM32G070KBT6, Package_QFP:LQFP-32_7x7mm_P0.8mm, symbol MCU_ST_STM32G0:STM32G071KxT
Connections:
- new net +3V3: C?.1, U?.4 (VDD/VDDA)
- new net GND: C?.2, U?.5 (VSS/VSSA)
Changed lines of the file:
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@@
 (kicad_sch (version 20211123) (generator eeschema)
   (paper "A4")
+  (junction (at 132.08 43.18) (diameter 0) (color 0 0 0 0)
+  )
+  (wire (pts (xy 143.51 58.42) (xy 143.51 43.18))
+    (stroke (width 0) (type default) (color 0 0 0 0))
+  )
+  (wire (pts (xy 132.08 43.18) (xy 132.08 46.99))
+    (stroke (width 0) (type default) (color 0 0 0 0))
+  )
+  (wire (pts (xy 124.46 43.18) (xy 132.08 43.18))
+    (stroke (width 0) (type default) (color 0 0 0 0))
+  )
+  (wire (pts (xy 143.51 114.3) (xy 143.51 116.84))
+    (stroke (width 0) (type default) (color 0 0 0 0))
+  )
+  (wire (pts (xy 143.51 43.18) (xy 132.08 43.18))
+    (stroke (width 0) (type default) (color 0 0 0 0))
+  )
+  (wire (pts (xy 132.08 52.07) (xy 132.08 55.88))
+    (stroke (width 0) (type default) (color 0 0 0 0))
+  )
+  (hierarchical_label "+3V3" (shape input) (at 124.46 43.18 180)
+    (effects (font (size 1.27 1.27)) (justify right))
+  )
+  (symbol (lib_id "Device:C_Small") (at 132.08 49.53 0) (unit 1)
+    (in_bom yes) (on_board yes) (fields_autoplaced)
+    (property "Reference" "C?" (id 0) (at 134.62 48.2662 0)
+      (effects (font (size 1.27 1.27)) (justify left))
+    )
+    (property "Value" "1uF" (id 1) (at 134.62 50.8062 0)
+      (effects (font (size 1.27 1.27)) (justify left))
+    )
+    (property "Footprint" "" (id 2) (at 132.08 49.53 0)
+      (effects (font (size 1.27 1.27)) hide)
+    )
+    (property "Datasheet" "~" (id 3) (at 132.08 49.53 0)
+      (effects (font (size 1.27 1.27)) hide)
+    )
+    (pin "1")
+    (pin "2")
+  )
+  (symbol (lib_id "power:GND") (at 143.51 116.84 0) (unit 1)
+    (in_bom yes) (on_board yes) (fields_autoplaced)
+    (property "Reference" "#PWR?" (id 0) (at 143.51 123.19 0)
+      (effects (font (size 1.27 1.27)) hide)
+    )
+    (property "Value" "GND" (id 1) (at 143.51 121.92 0)
+      (effects (font (size 1.27 1.27)) hide)
+    )
+    (property "Footprint" "" (id 2) (at 143.51 116.84 0)
+      (effects (font (size 1.27 1.27)) hide)
+    )
+    (property "Datasheet" "" (id 3) (at 143.51 116.84 0)
+      (effects (font (size 1.27 1.27)) hide)
+    )
+    (pin "1")
+  )
+  (symbol (lib_id "MCU_ST_STM32G0:STM32G071KxT") (at 143.51 86.36 0) (unit 1)
+    (in_bom yes) (on_board yes) (fields_autoplaced)
+    (property "Reference" "U?" (id 0) (at 145.5294 55.88 0)
+      (effects (font (size 1.27 1.27)) (justify left))
+    )
+    (property "Value" "STM32G070KBT6" (id 1) (at 145.5294 58.42 0)
+      (effects (font (size 1.27 1.27)) (justify left))
+    )
+    (property "Footprint" "Package_QFP:LQFP-32_7x7mm_P0.8mm" (id 2) (at 140.97 113.03 0)
+      (effects (font (size 1.27 1.27)) (justify right) hide)
+    )
+    (property "Datasheet" "https://www.st.com/resource/en/datasheet/stm32g071kb.pdf" (id 3) (at 143.51 86.36 0)
+      (effects (font (size 1.27 1.27)) hide)
+    )
+    (pin "1")
+    (pin "10")
+    (pin "11")
+    (pin "12")
+    (pin "13")
+    (pin "14")
+    (pin "15")
+    (pin "16")
+    (pin "17")
+    (pin "18")
+    (pin "19")
+    (pin "2")
+    (pin "20")
+    (pin "21")
+    (pin "22")
+    (pin "23")
+    (pin "24")
+    (pin "25")
+    (pin "26")
+    (pin "27")
+    (pin "28")
+    (pin "29")
+    (pin "3")
+    (pin "30")
+    (pin "31")
+    (pin "32")
+    (pin "4")
+    (pin "5")
+    (pin "6")
+    (pin "7")
+    (pin "8")
+    (pin "9")
+  )
+  (symbol (lib_id "power:GND") (at 132.08 55.88 0) (unit 1)
+    (in_bom yes) (on_board yes) (fields_autoplaced)
+    (property "Reference" "#PWR?" (id 0) (at 132.08 62.23 0)
+      (effects (font (size 1.27 1.27)) hide)
+    )
+    (property "Value" "GND" (id 1) (at 132.08 60.96 0)
+      (effects (font (size 1.27 1.27)) hide)
+    )
+    (property "Footprint" "" (id 2) (at 132.08 55.88 0)
+      (effects (font (size 1.27 1.27)) hide)
+    )
+    (property "Datasheet" "" (id 3) (at 132.08 55.88 0)
+      (effects (font (size 1.27 1.27)) hide)
+    )
+    (pin "1")
+  )
 )

Commit message: Updates
Updates
Connections:
- net RXD: now reaches U?.10 (PA3)
- net ~{FLASH_CS}: now reaches U?.11 (PA4)
- net FLASH_SCK: now reaches U?.12 (PA5)
- net FLASH_MISO: now reaches U?.13 (PA6)
- net FLASH_MOSI: now reaches U?.14 (PA7)
- net TXD: now reaches U?.9 (PA2)
Changed lines of the file:
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@@
+    (stroke (width 0) (type default) (color 0 0 0 0))
+  )
+  (wire (pts (xy 121.92 73.66) (xy 125.73 73.66))
+    (stroke (width 0) (type default) (color 0 0 0 0))
+  )
+  (wire (pts (xy 121.92 81.28) (xy 125.73 81.28))
+    (stroke (width 0) (type default) (color 0 0 0 0))
+  )
+  (wire (pts (xy 121.92 71.12) (xy 125.73 71.12))
     (stroke (width 0) (type default) (color 0 0 0 0))
   )
@@
     (stroke (width 0) (type default) (color 0 0 0 0))
   )
+  (wire (pts (xy 121.92 76.2) (xy 125.73 76.2))
+    (stroke (width 0) (type default) (color 0 0 0 0))
+  )
   (wire (pts (xy 143.51 43.18) (xy 132.08 43.18))
+    (stroke (width 0) (type default) (color 0 0 0 0))
+  )
+  (wire (pts (xy 121.92 78.74) (xy 125.73 78.74))
+    (stroke (width 0) (type default) (color 0 0 0 0))
+  )
+  (wire (pts (xy 121.92 83.82) (xy 125.73 83.82))
     (stroke (width 0) (type default) (color 0 0 0 0))
   )
@@
     (effects (font (size 1.27 1.27)) (justify right))
   )
+  (hierarchical_label "FLASH_SCK" (shape output) (at 121.92 78.74 180)
+    (effects (font (size 1.27 1.27)) (justify right))
+  )
+  (hierarchical_label "RXD" (shape input) (at 121.92 73.66 180)
+    (effects (font (size 1.27 1.27)) (justify right))
+  )
+  (hierarchical_label "FLASH_MISO" (shape input) (at 121.92 81.28 180)
+    (effects (font (size 1.27 1.27)) (justify right))
+  )
+  (hierarchical_label "~{FLASH_CS}" (shape output) (at 121.92 76.2 180)
+    (effects (font (size 1.27 1.27)) (justify right))
+  )
+  (hierarchical_label "FLASH_MOSI" (shape output) (at 121.92 83.82 180)
+    (effects (font (size 1.27 1.27)) (justify right))
+  )
+  (hierarchical_label "TXD" (shape output) (at 121.92 71.12 180)
+    (effects (font (size 1.27 1.27)) (justify right))
+  )

Commit message: More updates
Connections:
- net RXD: now also U?.21 (PA10); no longer U?.10 (PA3)
- net TXD: now also U?.19 (PA9); no longer U?.9 (PA2)
- net RMOTOR_FORWARD: now reaches U?.15 (PB0)
- net RMOTOR_BACKWARD: now reaches U?.16 (PB1)
- net LMOTOR_FORWARD: now reaches U?.28 (PB4)
- net LMOTOR_BACKWARD: now reaches U?.29 (PB5)
- net LMOTOR_PPM: now reaches U?.31 (PB7)
- net RMOTOR_PPM: now reaches U?.32 (PB8)
- net +TEMP_VSENSE: now reaches U?.7 (PA0)
- net +VBAT_VSENSE: now reaches U?.8 (PA1)
- new net +MOTOR_ISENSE: U?.9 (PA2)
- new net +XT_ISENSE: U?.10 (PA3)
Changed lines of the file:
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@@
-    (stroke (width 0) (type default) (color 0 0 0 0))
-  )
-  (wire (pts (xy 121.92 73.66) (xy 125.73 73.66))
     (stroke (width 0) (type default) (color 0 0 0 0))
   )
@@
     (stroke (width 0) (type default) (color 0 0 0 0))
   )
-  (wire (pts (xy 121.92 71.12) (xy 125.73 71.12))
+  (wire (pts (xy 121.92 88.9) (xy 125.73 88.9))
     (stroke (width 0) (type default) (color 0 0 0 0))
   )
   (wire (pts (xy 124.46 43.18) (xy 132.08 43.18))
+    (stroke (width 0) (type default) (color 0 0 0 0))
+  )
+  (wire (pts (xy 161.29 86.36) (xy 163.83 86.36))
+    (stroke (width 0) (type default) (color 0 0 0 0))
+  )
+  (wire (pts (xy 161.29 66.04) (xy 163.83 66.04))
+    (stroke (width 0) (type default) (color 0 0 0 0))
+  )
+  (wire (pts (xy 121.92 71.12) (xy 125.73 71.12))
     (stroke (width 0) (type default) (color 0 0 0 0))
   )
@@
     (stroke (width 0) (type default) (color 0 0 0 0))
   )
+  (wire (pts (xy 121.92 91.44) (xy 125.73 91.44))
+    (stroke (width 0) (type default) (color 0 0 0 0))
+  )
+  (wire (pts (xy 121.92 68.58) (xy 125.73 68.58))
+    (stroke (width 0) (type default) (color 0 0 0 0))
+  )
   (wire (pts (xy 143.51 43.18) (xy 132.08 43.18))
     (stroke (width 0) (type default) (color 0 0 0 0))
@@
     (stroke (width 0) (type default) (color 0 0 0 0))
   )
+  (wire (pts (xy 121.92 66.04) (xy 125.73 66.04))
+    (stroke (width 0) (type default) (color 0 0 0 0))
+  )
   (wire (pts (xy 121.92 83.82) (xy 125.73 83.82))
+    (stroke (width 0) (type default) (color 0 0 0 0))
+  )
+  (wire (pts (xy 161.29 68.58) (xy 163.83 68.58))
+    (stroke (width 0) (type default) (color 0 0 0 0))
+  )
+  (wire (pts (xy 121.92 73.66) (xy 125.73 73.66))
+    (stroke (width 0) (type default) (color 0 0 0 0))
+  )
+  (wire (pts (xy 161.29 76.2) (xy 163.83 76.2))
     (stroke (width 0) (type default) (color 0 0 0 0))
   )
@@
     (stroke (width 0) (type default) (color 0 0 0 0))
   )
+  (wire (pts (xy 161.29 83.82) (xy 163.83 83.82))
+    (stroke (width 0) (type default) (color 0 0 0 0))
+  )
+  (wire (pts (xy 161.29 78.74) (xy 163.83 78.74))
+    (stroke (width 0) (type default) (color 0 0 0 0))
+  )
+  (hierarchical_label "RMOTOR_PPM" (shape input) (at 163.83 86.36 0)
+    (effects (font (size 1.27 1.27)) (justify left))
+  )
+  (hierarchical_label "+VBAT_VSENSE" (shape input) (at 121.92 68.58 180)
+    (effects (font (size 1.27 1.27)) (justify right))
+  )
+  (hierarchical_label "LMOTOR_PPM" (shape input) (at 163.83 83.82 0)
+    (effects (font (size 1.27 1.27)) (justify left))
+  )
+  (hierarchical_label "RMOTOR_BACKWARD" (shape output) (at 163.83 68.58 0)
+    (effects (font (size 1.27 1.27)) (justify left))
+  )
   (hierarchical_label "+3V3" (shape input) (at 124.46 43.18 180)
     (effects (font (size 1.27 1.27)) (justify right))
+  )
+  (hierarchical_label "+XT_ISENSE" (shape input) (at 121.92 73.66 180)
+    (effects (font (size 1.27 1.27)) (justify right))
+  )
+  (hierarchical_label "LMOTOR_FORWARD" (shape output) (at 163.83 76.2 0)
+    (effects (font (size 1.27 1.27)) (justify left))
   )
   (hierarchical_label "FLASH_SCK" (shape output) (at 121.92 78.74 180)
     (effects (font (size 1.27 1.27)) (justify right))
   )
-  (hierarchical_label "RXD" (shape input) (at 121.92 73.66 180)
+  (hierarchical_label "RXD" (shape input) (at 121.92 91.44 180)
     (effects (font (size 1.27 1.27)) (justify right))
   )
@@
     (effects (font (size 1.27 1.27)) (justify right))
   )
+  (hierarchical_label "+TEMP_VSENSE" (shape input) (at 121.92 66.04 180)
+    (effects (font (size 1.27 1.27)) (justify right))
+  )
+  (hierarchical_label "+MOTOR_ISENSE" (shape input) (at 121.92 71.12 180)
+    (effects (font (size 1.27 1.27)) (justify right))
+  )
+  (hierarchical_label "LMOTOR_BACKWARD" (shape output) (at 163.83 78.74 0)
+    (effects (font (size 1.27 1.27)) (justify left))
+  )
+  (hierarchical_label "RMOTOR_FORWARD" (shape output) (at 163.83 66.04 0)
+    (effects (font (size 1.27 1.27)) (justify left))
+  )
   (hierarchical_label "FLASH_MOSI" (shape output) (at 121.92 83.82 180)
     (effects (font (size 1.27 1.27)) (justify right))
   )
-  (hierarchical_label "TXD" (shape output) (at 121.92 71.12 180)
+  (hierarchical_label "TXD" (shape output) (at 121.92 88.9 180)
     (effects (font (size 1.27 1.27)) (justify right))
   )

Commit message: Updates
Parts:
- C14: renamed from C?; footprint (none) -> Capacitor_SMD:C_0603_1608Metric; MPN (none) -> CC0603KRX5R8BB105
- U8: renamed from U?; MPN (none) -> STM32G070KBT6
Connections:
- net SWDIO: now reaches U8.24 (PA13)
- net SWCLK: now reaches U8.25 (PA14/BOOT0)
Changed lines of the file:
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@@
+    (stroke (width 0) (type default) (color 0 0 0 0))
+  )
+  (wire (pts (xy 121.92 91.44) (xy 125.73 91.44))
     (stroke (width 0) (type default) (color 0 0 0 0))
   )
@@
     (stroke (width 0) (type default) (color 0 0 0 0))
   )
+  (wire (pts (xy 124.46 43.18) (xy 132.08 43.18))
+    (stroke (width 0) (type default) (color 0 0 0 0))
+  )
+  (wire (pts (xy 161.29 86.36) (xy 163.83 86.36))
+    (stroke (width 0) (type default) (color 0 0 0 0))
+  )
+  (wire (pts (xy 121.92 99.06) (xy 125.73 99.06))
+    (stroke (width 0) (type default) (color 0 0 0 0))
+  )
   (wire (pts (xy 121.92 88.9) (xy 125.73 88.9))
     (stroke (width 0) (type default) (color 0 0 0 0))
   )
-  (wire (pts (xy 124.46 43.18) (xy 132.08 43.18))
-    (stroke (width 0) (type default) (color 0 0 0 0))
-  )
-  (wire (pts (xy 161.29 86.36) (xy 163.83 86.36))
-    (stroke (width 0) (type default) (color 0 0 0 0))
-  )
   (wire (pts (xy 161.29 66.04) (xy 163.83 66.04))
     (stroke (width 0) (type default) (color 0 0 0 0))
@@
     (stroke (width 0) (type default) (color 0 0 0 0))
   )
-  (wire (pts (xy 121.92 91.44) (xy 125.73 91.44))
-    (stroke (width 0) (type default) (color 0 0 0 0))
-  )
   (wire (pts (xy 121.92 68.58) (xy 125.73 68.58))
     (stroke (width 0) (type default) (color 0 0 0 0))
@@
     (stroke (width 0) (type default) (color 0 0 0 0))
   )
+  (wire (pts (xy 121.92 101.6) (xy 125.73 101.6))
+    (stroke (width 0) (type default) (color 0 0 0 0))
+  )
   (wire (pts (xy 161.29 76.2) (xy 163.83 76.2))
     (stroke (width 0) (type default) (color 0 0 0 0))
@@
     (effects (font (size 1.27 1.27)) (justify right))
   )
+  (hierarchical_label "SWDIO" (shape bidirectional) (at 121.92 99.06 180)
+    (effects (font (size 1.27 1.27)) (justify right))
+  )
   (hierarchical_label "+XT_ISENSE" (shape input) (at 121.92 73.66 180)
     (effects (font (size 1.27 1.27)) (justify right))
@@
     (effects (font (size 1.27 1.27)) (justify left))
   )
+  (hierarchical_label "SWCLK" (shape input) (at 121.92 101.6 180)
+    (effects (font (size 1.27 1.27)) (justify right))
+  )
   (hierarchical_label "FLASH_MOSI" (shape output) (at 121.92 83.82 180)
     (effects (font (size 1.27 1.27)) (justify right))
@@
   (symbol (lib_id "Device:C_Small") (at 132.08 49.53 0) (unit 1)
     (in_bom yes) (on_board yes) (fields_autoplaced)
-    (property "Reference" "C?" (id 0) (at 134.62 48.2662 0)
+    (property "Reference" "C14" (id 0) (at 134.62 48.2662 0)
       (effects (font (size 1.27 1.27)) (justify left))
     )
@@
       (effects (font (size 1.27 1.27)) (justify left))
     )
-    (property "Footprint" "" (id 2) (at 132.08 49.53 0)
+    (property "Footprint" "Capacitor_SMD:C_0603_1608Metric" (id 2) (at 132.08 49.53 0)
       (effects (font (size 1.27 1.27)) hide)
     )
     (property "Datasheet" "~" (id 3) (at 132.08 49.53 0)
+      (effects (font (size 1.27 1.27)) hide)
+    )
+    (property "MPN" "CC0603KRX5R8BB105" (id 4) (at 132.08 49.53 0)
       (effects (font (size 1.27 1.27)) hide)
     )
@@
   (symbol (lib_id "power:GND") (at 143.51 116.84 0) (unit 1)
     (in_bom yes) (on_board yes) (fields_autoplaced)
-    (property "Reference" "#PWR?" (id 0) (at 143.51 123.19 0)
+    (property "Reference" "#PWR027" (id 0) (at 143.51 123.19 0)
       (effects (font (size 1.27 1.27)) hide)
     )
@@
   (symbol (lib_id "MCU_ST_STM32G0:STM32G071KxT") (at 143.51 86.36 0) (unit 1)
     (in_bom yes) (on_board yes) (fields_autoplaced)
-    (property "Reference" "U?" (id 0) (at 145.5294 55.88 0)
+    (property "Reference" "U8" (id 0) (at 145.5294 55.88 0)
       (effects (font (size 1.27 1.27)) (justify left))
     )
@@
     )
     (property "Datasheet" "https://www.st.com/resource/en/datasheet/stm32g071kb.pdf" (id 3) (at 143.51 86.36 0)
+      (effects (font (size 1.27 1.27)) hide)
+    )
+    (property "MPN" "STM32G070KBT6" (id 4) (at 143.51 86.36 0)
       (effects (font (size 1.27 1.27)) hide)
     )
@@
   (symbol (lib_id "power:GND") (at 132.08 55.88 0) (unit 1)
     (in_bom yes) (on_board yes) (fields_autoplaced)
-    (property "Reference" "#PWR?" (id 0) (at 132.08 62.23 0)
-      (effects (font (size 1.27 1.27)) hide)
-    )
+    (property "Reference" "#PWR026" (id 0) (at 132.08 62.23 0)
+      (effects (font (size 1.27 1.27)) hide)
+    )

Commit message: So many updates
Parts:
- C14: footprint Capacitor_SMD:C_0603_1608Metric -> Capacitor_SMD:C_0402_1005Metric; MPN CC0603KRX5R8BB105 -> CC0402KRX5R8BB105
Connections:
- net LMOTOR_FORWARD: now also U8.30 (PB6); no longer U8.28 (PB4)
- net RMOTOR_BACKWARD: now also U8.28 (PB4); no longer U8.16 (PB1)
- net RMOTOR_FORWARD: now also U8.27 (PB3); no longer U8.15 (PB0)
- net +MOTOR_ISENSE renamed +RMOTOR_ISENSE
- net +TEMP_VSENSE renamed +LTEMP_VSENSE
- net +LTEMP_VSENSE: now also U8.15 (PB0)
- new net +RTEMP_VSENSE: U8.16 (PB1)
- no-connect marks 0 -> 8
Changed lines of the file:
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@@
   (junction (at 132.08 43.18) (diameter 0) (color 0 0 0 0)
   )
+  (no_connect (at 125.73 93.98))
+  (no_connect (at 125.73 96.52))
+  (no_connect (at 125.73 104.14))
+  (no_connect (at 161.29 99.06))
+  (no_connect (at 161.29 96.52))
+  (no_connect (at 161.29 93.98))
+  (no_connect (at 161.29 88.9))
+  (no_connect (at 161.29 71.12))
   (wire (pts (xy 143.51 58.42) (xy 143.51 43.18))
     (stroke (width 0) (type default) (color 0 0 0 0))
   )
   (wire (pts (xy 132.08 43.18) (xy 132.08 46.99))
+    (stroke (width 0) (type default) (color 0 0 0 0))
+  )
+  (wire (pts (xy 161.29 81.28) (xy 163.83 81.28))
+    (stroke (width 0) (type default) (color 0 0 0 0))
+  )
+  (wire (pts (xy 161.29 73.66) (xy 163.83 73.66))
     (stroke (width 0) (type default) (color 0 0 0 0))
   )
@@
     (stroke (width 0) (type default) (color 0 0 0 0))
   )
-  (wire (pts (xy 161.29 66.04) (xy 163.83 66.04))
-    (stroke (width 0) (type default) (color 0 0 0 0))
-  )
   (wire (pts (xy 121.92 71.12) (xy 125.73 71.12))
     (stroke (width 0) (type default) (color 0 0 0 0))
@@
     (stroke (width 0) (type default) (color 0 0 0 0))
   )
+  (wire (pts (xy 161.29 66.04) (xy 163.83 66.04))
+    (stroke (width 0) (type default) (color 0 0 0 0))
+  )
   (wire (pts (xy 143.51 43.18) (xy 132.08 43.18))
+    (stroke (width 0) (type default) (color 0 0 0 0))
+  )
+  (wire (pts (xy 161.29 76.2) (xy 163.83 76.2))
+    (stroke (width 0) (type default) (color 0 0 0 0))
+  )
+  (wire (pts (xy 161.29 68.58) (xy 163.83 68.58))
     (stroke (width 0) (type default) (color 0 0 0 0))
   )
@@
     (stroke (width 0) (type default) (color 0 0 0 0))
   )
-  (wire (pts (xy 161.29 68.58) (xy 163.83 68.58))
-    (stroke (width 0) (type default) (color 0 0 0 0))
-  )
   (wire (pts (xy 121.92 73.66) (xy 125.73 73.66))
     (stroke (width 0) (type default) (color 0 0 0 0))
   )
   (wire (pts (xy 121.92 101.6) (xy 125.73 101.6))
-    (stroke (width 0) (type default) (color 0 0 0 0))
-  )
-  (wire (pts (xy 161.29 76.2) (xy 163.83 76.2))
     (stroke (width 0) (type default) (color 0 0 0 0))
   )
@@
     (stroke (width 0) (type default) (color 0 0 0 0))
   )
+  (hierarchical_label "+RTEMP_VSENSE" (shape input) (at 163.83 68.58 0)
+    (effects (font (size 1.27 1.27)) (justify left))
+  )
   (hierarchical_label "RMOTOR_PPM" (shape input) (at 163.83 86.36 0)
     (effects (font (size 1.27 1.27)) (justify left))
+  )
+  (hierarchical_label "+RMOTOR_ISENSE" (shape input) (at 121.92 71.12 180)
+    (effects (font (size 1.27 1.27)) (justify right))
   )
   (hierarchical_label "+VBAT_VSENSE" (shape input) (at 121.92 68.58 180)
@@
     (effects (font (size 1.27 1.27)) (justify left))
   )
-  (hierarchical_label "RMOTOR_BACKWARD" (shape output) (at 163.83 68.58 0)
+  (hierarchical_label "RMOTOR_BACKWARD" (shape output) (at 163.83 76.2 0)
     (effects (font (size 1.27 1.27)) (justify left))
   )
@@
     (effects (font (size 1.27 1.27)) (justify right))
   )
-  (hierarchical_label "LMOTOR_FORWARD" (shape output) (at 163.83 76.2 0)
+  (hierarchical_label "LMOTOR_FORWARD" (shape output) (at 163.83 81.28 0)
     (effects (font (size 1.27 1.27)) (justify left))
   )
@@
     (effects (font (size 1.27 1.27)) (justify right))
   )
-  (hierarchical_label "+TEMP_VSENSE" (shape input) (at 121.92 66.04 180)
-    (effects (font (size 1.27 1.27)) (justify right))
-  )
-  (hierarchical_label "+MOTOR_ISENSE" (shape input) (at 121.92 71.12 180)
+  (hierarchical_label "+LTEMP_VSENSE" (shape input) (at 121.92 66.04 180)
     (effects (font (size 1.27 1.27)) (justify right))
   )
@@
     (effects (font (size 1.27 1.27)) (justify left))
   )
-  (hierarchical_label "RMOTOR_FORWARD" (shape output) (at 163.83 66.04 0)
+  (hierarchical_label "RMOTOR_FORWARD" (shape output) (at 163.83 73.66 0)
     (effects (font (size 1.27 1.27)) (justify left))
   )
@@
     (effects (font (size 1.27 1.27)) (justify right))
   )
+  (hierarchical_label "+LTEMP_VSENSE" (shape input) (at 163.83 66.04 0)
+    (effects (font (size 1.27 1.27)) (justify left))
+  )
   (symbol (lib_id "Device:C_Small") (at 132.08 49.53 0) (unit 1)
     (in_bom yes) (on_board yes) (fields_autoplaced)
@@
       (effects (font (size 1.27 1.27)) (justify left))
     )
-    (property "Footprint" "Capacitor_SMD:C_0603_1608Metric" (id 2) (at 132.08 49.53 0)
+    (property "Footprint" "Capacitor_SMD:C_0402_1005Metric" (id 2) (at 132.08 49.53 0)
       (effects (font (size 1.27 1.27)) hide)
     )
@@
       (effects (font (size 1.27 1.27)) hide)
     )
-    (property "MPN" "CC0603KRX5R8BB105" (id 4) (at 132.08 49.53 0)
+    (property "MPN" "CC0402KRX5R8BB105" (id 4) (at 132.08 49.53 0)
       (effects (font (size 1.27 1.27)) hide)
     )
