File: MotorController/MCU.kicad_sch (KiCad schematic)
At the start: 2 parts, among them U8 STM32G070KBT6

Commit message: my god
my god
Connections:
- net +LTEMP_VSENSE: no longer U8.15 (PB0)
- net LMOTOR_PPM: now also U8.32 (PB8); no longer U8.31 (PB7)
- net RMOTOR_PPM: now also U8.31 (PB7); no longer U8.32 (PB8)
- new net +LMOTOR_ISENSE: U8.15 (PB0)
- no-connect marks 8 -> 9
Changed lines of the file:
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@@
   (junction (at 132.08 43.18) (diameter 0) (color 0 0 0 0)
   )
+  (no_connect (at 125.73 86.36))
   (no_connect (at 125.73 93.98))
   (no_connect (at 125.73 96.52))
@@
     (stroke (width 0) (type default) (color 0 0 0 0))
   )
-  (wire (pts (xy 161.29 86.36) (xy 163.83 86.36))
-    (stroke (width 0) (type default) (color 0 0 0 0))
-  )
   (wire (pts (xy 121.92 99.06) (xy 125.73 99.06))
     (stroke (width 0) (type default) (color 0 0 0 0))
@@
   )
   (wire (pts (xy 121.92 71.12) (xy 125.73 71.12))
+    (stroke (width 0) (type default) (color 0 0 0 0))
+  )
+  (wire (pts (xy 161.29 83.82) (xy 163.83 83.82))
     (stroke (width 0) (type default) (color 0 0 0 0))
   )
@@
     (stroke (width 0) (type default) (color 0 0 0 0))
   )
+  (wire (pts (xy 161.29 86.36) (xy 163.83 86.36))
+    (stroke (width 0) (type default) (color 0 0 0 0))
+  )
   (wire (pts (xy 121.92 73.66) (xy 125.73 73.66))
     (stroke (width 0) (type default) (color 0 0 0 0))
@@
     (stroke (width 0) (type default) (color 0 0 0 0))
   )
-  (wire (pts (xy 161.29 83.82) (xy 163.83 83.82))
-    (stroke (width 0) (type default) (color 0 0 0 0))
-  )
   (wire (pts (xy 161.29 78.74) (xy 163.83 78.74))
     (stroke (width 0) (type default) (color 0 0 0 0))
@@
     (effects (font (size 1.27 1.27)) (justify left))
   )
-  (hierarchical_label "RMOTOR_PPM" (shape input) (at 163.83 86.36 0)
+  (hierarchical_label "RMOTOR_PPM" (shape input) (at 163.83 83.82 0)
     (effects (font (size 1.27 1.27)) (justify left))
   )
@@
     (effects (font (size 1.27 1.27)) (justify right))
   )
-  (hierarchical_label "LMOTOR_PPM" (shape input) (at 163.83 83.82 0)
+  (hierarchical_label "LMOTOR_PPM" (shape input) (at 163.83 86.36 0)
     (effects (font (size 1.27 1.27)) (justify left))
   )
@@
     (effects (font (size 1.27 1.27)) (justify right))
   )
+  (hierarchical_label "+LMOTOR_ISENSE" (shape input) (at 163.83 66.04 0)
+    (effects (font (size 1.27 1.27)) (justify left))
+  )
   (hierarchical_label "~{FLASH_CS}" (shape output) (at 121.92 76.2 180)
     (effects (font (size 1.27 1.27)) (justify right))
@@
     (effects (font (size 1.27 1.27)) (justify right))
   )
-  (hierarchical_label "+LTEMP_VSENSE" (shape input) (at 163.83 66.04 0)
-    (effects (font (size 1.27 1.27)) (justify left))
-  )
   (symbol (lib_id "Device:C_Small") (at 132.08 49.53 0) (unit 1)

Commit message: ahhhhh
Connections:
- net +LMOTOR_ISENSE: now also U8.9 (PA2); no longer U8.15 (PB0)
- net +RMOTOR_ISENSE: now also U8.15 (PB0); no longer U8.9 (PA2)
- net RMOTOR_BACKWARD: now also U8.27 (PB3); no longer U8.28 (PB4)
- net RMOTOR_FORWARD: now also U8.28 (PB4); no longer U8.27 (PB3)
Changed lines of the file:
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@@
-    (stroke (width 0) (type default) (color 0 0 0 0))
-  )
-  (wire (pts (xy 161.29 81.28) (xy 163.83 81.28))
-    (stroke (width 0) (type default) (color 0 0 0 0))
-  )
-  (wire (pts (xy 161.29 73.66) (xy 163.83 73.66))
     (stroke (width 0) (type default) (color 0 0 0 0))
   )
@@
     (stroke (width 0) (type default) (color 0 0 0 0))
   )
+  (wire (pts (xy 161.29 76.2) (xy 163.83 76.2))
+    (stroke (width 0) (type default) (color 0 0 0 0))
+  )
   (wire (pts (xy 121.92 99.06) (xy 125.73 99.06))
     (stroke (width 0) (type default) (color 0 0 0 0))
@@
     (stroke (width 0) (type default) (color 0 0 0 0))
   )
-  (wire (pts (xy 121.92 71.12) (xy 125.73 71.12))
+  (wire (pts (xy 161.29 83.82) (xy 163.83 83.82))
     (stroke (width 0) (type default) (color 0 0 0 0))
   )
-  (wire (pts (xy 161.29 83.82) (xy 163.83 83.82))
+  (wire (pts (xy 161.29 73.66) (xy 163.83 73.66))
     (stroke (width 0) (type default) (color 0 0 0 0))
   )
@@
     (stroke (width 0) (type default) (color 0 0 0 0))
   )
-  (wire (pts (xy 161.29 66.04) (xy 163.83 66.04))
-    (stroke (width 0) (type default) (color 0 0 0 0))
-  )
   (wire (pts (xy 143.51 43.18) (xy 132.08 43.18))
     (stroke (width 0) (type default) (color 0 0 0 0))
   )
-  (wire (pts (xy 161.29 76.2) (xy 163.83 76.2))
+  (wire (pts (xy 161.29 81.28) (xy 163.83 81.28))
     (stroke (width 0) (type default) (color 0 0 0 0))
   )
   (wire (pts (xy 161.29 68.58) (xy 163.83 68.58))
+    (stroke (width 0) (type default) (color 0 0 0 0))
+  )
+  (wire (pts (xy 161.29 78.74) (xy 163.83 78.74))
     (stroke (width 0) (type default) (color 0 0 0 0))
   )
@@
     (stroke (width 0) (type default) (color 0 0 0 0))
   )
+  (wire (pts (xy 121.92 71.12) (xy 125.73 71.12))
+    (stroke (width 0) (type default) (color 0 0 0 0))
+  )
   (wire (pts (xy 161.29 86.36) (xy 163.83 86.36))
     (stroke (width 0) (type default) (color 0 0 0 0))
   )
   (wire (pts (xy 121.92 73.66) (xy 125.73 73.66))
+    (stroke (width 0) (type default) (color 0 0 0 0))
+  )
+  (wire (pts (xy 161.29 66.04) (xy 163.83 66.04))
     (stroke (width 0) (type default) (color 0 0 0 0))
   )
@@
     (stroke (width 0) (type default) (color 0 0 0 0))
   )
-  (wire (pts (xy 161.29 78.74) (xy 163.83 78.74))
-    (stroke (width 0) (type default) (color 0 0 0 0))
-  )
   (hierarchical_label "+RTEMP_VSENSE" (shape input) (at 163.83 68.58 0)
     (effects (font (size 1.27 1.27)) (justify left))
@@
     (effects (font (size 1.27 1.27)) (justify left))
   )
-  (hierarchical_label "+RMOTOR_ISENSE" (shape input) (at 121.92 71.12 180)
-    (effects (font (size 1.27 1.27)) (justify right))
+  (hierarchical_label "+RMOTOR_ISENSE" (shape input) (at 163.83 66.04 0)
+    (effects (font (size 1.27 1.27)) (justify left))
   )
   (hierarchical_label "+VBAT_VSENSE" (shape input) (at 121.92 68.58 180)
@@
     (effects (font (size 1.27 1.27)) (justify left))
   )
-  (hierarchical_label "RMOTOR_BACKWARD" (shape output) (at 163.83 76.2 0)
+  (hierarchical_label "RMOTOR_BACKWARD" (shape output) (at 163.83 73.66 0)
     (effects (font (size 1.27 1.27)) (justify left))
   )
@@
     (effects (font (size 1.27 1.27)) (justify right))
   )
-  (hierarchical_label "+LMOTOR_ISENSE" (shape input) (at 163.83 66.04 0)
-    (effects (font (size 1.27 1.27)) (justify left))
+  (hierarchical_label "+LMOTOR_ISENSE" (shape input) (at 121.92 71.12 180)
+    (effects (font (size 1.27 1.27)) (justify right))
   )
   (hierarchical_label "~{FLASH_CS}" (shape output) (at 121.92 76.2 180)
@@
     (effects (font (size 1.27 1.27)) (justify left))
   )
-  (hierarchical_label "RMOTOR_FORWARD" (shape output) (at 163.83 73.66 0)
+  (hierarchical_label "RMOTOR_FORWARD" (shape output) (at 163.83 76.2 0)
     (effects (font (size 1.27 1.27)) (justify left))
   )
