File: MotorController/MotorController.kicad_pcb (KiCad board)
At the start: 2 copper layers, 50.8 x 19 mm, 89 parts, among them J1 Conn_01x02, J2 Conn_01x02, J3 Conn_01x03, J4 USB_B_Micro, J5 Conn_01x04, M1 Motor_DC, M2 Motor_DC, Q1 Q_NMOS_GDS, Q2 Q_NMOS_GDS, Q3 Q_NMOS_GDS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

Commit message: Changes
Changes
Parts:
- added D1: D_Small_Filled, Diode_SMD:D_SMA, F.Cu at (39.4, 25.7)
- added D10: GREEN, LED_SMD:LED_0603_1608Metric, F.Cu at (48.1, 30.4)
- added D11: D_Small_Filled, Diode_SMD:D_SOD-323, F.Cu at (47.4, 50.5)
- added D12: D_Small_Filled, Diode_SMD:D_SOD-323, F.Cu at (41.1, 56.1)
- added D13: D_Small_Filled, Diode_SMD:D_SOD-323, F.Cu at (37.9, 62.4)
- added D18: D_Small_Filled, Diode_SMD:D_SOD-323, F.Cu at (84.4, 30.4)
- added D19: D_Small_Filled, Diode_SMD:D_SOD-323, F.Cu at (90.7, 24.9)
- added D20: D_Small_Filled, Diode_SMD:D_SOD-323, F.Cu at (84.4, 33.4)
- added D21: D_Small_Filled, Diode_SMD:D_SOD-323, F.Cu at (81.3, 36.7)
- added D4: GREEN, LED_SMD:LED_0603_1608Metric, F.Cu at (36.8, 42.7)
- added D5: D_Small_Filled, Diode_SMD:D_SOD-323, F.Cu at (41.1, 59.0)
- added R34: 680, Resistor_SMD:R_0402_1005Metric, F.Cu at (40.2, 44.9)
- added R35: 680, Resistor_SMD:R_0402_1005Metric, F.Cu at (36.2, 45.0)
- Q1, Q2, Q3, Q4, Q5, Q6, Q7, Q8: value Q_NMOS_GDS -> SSM6K513NU-LF
- moved R3 98.8 mm to (45.9, 38.7)
- moved D3 96.7 mm to (38.2, 35.3)
- moved R1 93.0 mm to (47.1, 36.2)
- moved U8 91.6 mm to (69.1, 54.8)
- moved R6 89.4 mm to (44.8, 43.7)
- moved C24 89.2 mm to (99.0, 24.6)
- moved C8 87.6 mm to (49.9, 38.7)
- moved C2 86.3 mm to (51.2, 33.5)
- moved R5 85.3 mm to (47.1, 33.7)
- moved C23 83.9 mm to (90.6, 27.6)
- moved R21 82.6 mm to (96.8, 28.3)
- moved R9 81.0 mm to (38.0, 30.8)
- moved U2 80.9 mm to (50.7, 25.3)
- moved R10 78.6 mm to (40.8, 42.7)
- moved C14 76.4 mm to (76.8, 50.3)
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Connections:
- Q1 pad 1: Net-(D4-Pad2) -> +MOTOR_VBAT
- Q1 pad 3: Net-(C16-Pad2) -> Net-(Q1-Pad3)
- Q1 pad 4: (no net) -> Net-(C16-Pad2)
- Q1 pad 5: (no net) -> +MOTOR_VBAT
- Q1 pad 6: (no net) -> +MOTOR_VBAT
- Q1 pad 7: (no net) -> +MOTOR_VBAT
- Q1 pad 8: (no net) -> Net-(C16-Pad2)
- Q2 pad 1: Net-(D5-Pad2) -> Net-(C16-Pad2)
- Q2 pad 3: GND -> Net-(D5-Pad2)
- Q2 pad 4: (no net) -> GND
- Q2 pad 5: (no net) -> Net-(C16-Pad2)
- Q2 pad 6: (no net) -> Net-(C16-Pad2)
- Q2 pad 7: (no net) -> Net-(C16-Pad2)
- Q2 pad 8: (no net) -> GND
- Q3 pad 1: Net-(D10-Pad2) -> +MOTOR_VBAT
- Q3 pad 3: Net-(C18-Pad2) -> Net-(Q3-Pad3)
- Q3 pad 4: (no net) -> Net-(C18-Pad2)
- Q3 pad 5: (no net) -> +MOTOR_VBAT
- Q3 pad 6: (no net) -> +MOTOR_VBAT
- Q3 pad 7: (no net) -> +MOTOR_VBAT
- Q3 pad 8: (no net) -> Net-(C18-Pad2)
- Q4 pad 1: Net-(D11-Pad2) -> Net-(C18-Pad2)
- Q4 pad 3: GND -> Net-(Q4-Pad3)
- Q4 pad 4: (no net) -> GND
- Q4 pad 5: (no net) -> Net-(C18-Pad2)
- Q4 pad 6: (no net) -> Net-(C18-Pad2)
- Q4 pad 7: (no net) -> Net-(C18-Pad2)
- Q4 pad 8: (no net) -> GND
- Q5 pad 1: Net-(D12-Pad2) -> +MOTOR_VBAT
- Q5 pad 3: Net-(C21-Pad2) -> Net-(Q5-Pad3)
- Q5 pad 4: (no net) -> Net-(C21-Pad2)
- Q5 pad 5: (no net) -> +MOTOR_VBAT
- Q5 pad 6: (no net) -> +MOTOR_VBAT
- Q5 pad 7: (no net) -> +MOTOR_VBAT
- Q5 pad 8: (no net) -> Net-(C21-Pad2)
- Q6 pad 1: Net-(D13-Pad2) -> Net-(C21-Pad2)
- Q6 pad 3: GND -> Net-(Q6-Pad3)
- Q6 pad 4: (no net) -> GND
- Q6 pad 5: (no net) -> Net-(C21-Pad2)
- Q6 pad 6: (no net) -> Net-(C21-Pad2)
- Q6 pad 7: (no net) -> Net-(C21-Pad2)
- Q6 pad 8: (no net) -> GND
- Q7 pad 1: Net-(D18-Pad2) -> +MOTOR_VBAT
- Q7 pad 3: Net-(C23-Pad2) -> Net-(Q7-Pad3)
- Q7 pad 4: (no net) -> Net-(C23-Pad2)
- Q7 pad 5: (no net) -> +MOTOR_VBAT
- Q7 pad 6: (no net) -> +MOTOR_VBAT
- Q7 pad 7: (no net) -> +MOTOR_VBAT
- Q7 pad 8: (no net) -> Net-(C23-Pad2)
- Q8 pad 1: Net-(D19-Pad2) -> Net-(C23-Pad2)
- Q8 pad 3: GND -> Net-(Q8-Pad3)
- Q8 pad 4: (no net) -> GND
- Q8 pad 5: (no net) -> Net-(C23-Pad2)
- Q8 pad 6: (no net) -> Net-(C23-Pad2)
- Q8 pad 7: (no net) -> Net-(C23-Pad2)
- Q8 pad 8: (no net) -> GND
- R17 pad 1: Net-(D4-Pad2) -> Net-(Q1-Pad3)
- R19 pad 1: Net-(D10-Pad2) -> Net-(Q3-Pad3)
- R20 pad 2: Net-(D11-Pad2) -> Net-(Q4-Pad3)
- R24 pad 1: Net-(D12-Pad2) -> Net-(Q5-Pad3)
- R25 pad 2: Net-(D13-Pad2) -> Net-(Q6-Pad3)
- R26 pad 1: Net-(D18-Pad2) -> Net-(Q7-Pad3)
- R27 pad 2: Net-(D19-Pad2) -> Net-(Q8-Pad3)

Commit message: So many updates
Parts:
- added C26: 1uF, Capacitor_SMD:C_0402_1005Metric, F.Cu at (53.0, 43.3)
- added C27: DNU, Capacitor_SMD:C_0402_1005Metric, F.Cu at (57.0, 43.3)
- added C28: 0.1uF, Capacitor_SMD:C_0402_1005Metric, F.Cu at (163.8, 47.3)
- added C29: 680pF, Capacitor_SMD:C_0402_1005Metric, F.Cu at (161.9, 52.0)
- added D14: D_Small_Filled, Diode_SMD:D_SOD-323, B.Cu at (138.3, 81.7)
- added D15: D_Small_Filled, Footprints:TO-277B, B.Cu at (145.4, 81.0)
- added D16: D_Small_Filled, Diode_SMD:D_SOD-323, B.Cu at (138.3, 78.4)
- added D17: D_Small_Filled, Footprints:TO-277B, B.Cu at (149.9, 79.6)
- added D6: GREEN, LED_SMD:LED_0603_1608Metric, F.Cu at (151.4, 57.2)
- added D7: D_Small_Filled, Diode_SMD:D_SOD-323, B.Cu at (115.8, 78.0)
- added D8: D_Small_Filled, Footprints:TO-277B, B.Cu at (104.0, 79.6)
- added D9: D_Small_Filled, Footprints:TO-277B, B.Cu at (108.8, 81.0)
- added R36: 0, Resistor_SMD:R_0402_1005Metric, F.Cu at (47.9, 45.2)
- added R37: 0.2mOhms, Footprints:RES_WSK12161L000FEA, F.Cu at (48.4, 41.1)
- added R38: 0, Resistor_SMD:R_0402_1005Metric, F.Cu at (57.3, 39.5)
- added R39: 100, Resistor_SMD:R_0402_1005Metric, F.Cu at (159.0, 52.0)
- added U14: INA280A3IDCKR, Package_TO_SOT_SMD:SOT-353_SC-70-5, F.Cu at (53.1, 40.1)
- added U15: TMP236AQDBZRQ1, Package_TO_SOT_SMD:SC-59, F.Cu at (159.9, 48.7)
- C10, C11, C12, C13, C14, C2, C25, C3, C4, C6, C7, C8, C9: footprint Capacitor_SMD:C_0603_1608Metric -> Capacitor_SMD:C_0402_1005Metric
- C15, C19, C20, C24: footprint Capacitor_SMD:C_0603_1608Metric -> Capacitor_SMD:C_0402_1005Metric; moved to B.Cu
- C16, C18, C21, C23: value 40nF -> 33nF; footprint Capacitor_SMD:C_0603_1608Metric -> Capacitor_SMD:C_0402_1005Metric; moved to B.Cu
- C17, C22: footprint Capacitor_SMD:CP_Elec_10x10 -> Connector_PinHeader_2.54mm:PinHeader_1x02_P2.54mm_Vertical; moved to B.Cu
- D10: value GREEN -> D_Small_Filled; footprint LED_SMD:LED_0603_1608Metric -> Footprints:TO-277B; moved to B.Cu
- D11, D18, D19: footprint Diode_SMD:D_SOD-323 -> Footprints:TO-277B; moved to B.Cu
- D12, D13, D20, D21, D5, M2, Q1, Q2, Q3, Q4, Q5, Q6, Q7, Q8, U10, U11, U12, U9: moved to B.Cu
- R1, R10, R11, R12, R13, R2, R28, R29, R3, R30, R31, R32, R33, R5, R6, R7, R8: footprint Resistor_SMD:R_0603_1608Metric -> Resistor_SMD:R_0402_1005Metric
- R14, R15, R16, R17, R18, R19, R20, R21, R22, R23, R24, R25, R26, R27: footprint Resistor_SMD:R_0603_1608Metric -> Resistor_SMD:R_0402_1005Metric; moved to B.Cu
- moved D4 132.4 mm to (165.8, 72.4), turned to 90 degrees
- moved D1 131.2 mm to (162.7, 70.7), turned to -90 degrees
- moved U4 130.7 mm to (157.1, 70.5), turned to -90 degrees
- moved L1 130.5 mm to (157.3, 60.3), turned to 180 degrees
- moved U1 128.5 mm to (163.2, 64.9), turned to 90 degrees
- moved R34 128.0 mm to (165.7, 70.3), turned to 180 degrees
- moved R6 123.2 mm to (165.7, 67.6), turned to 180 degrees
- moved D2 122.1 mm to (161.7, 60.4), turned to 90 degrees
- moved R7 120.5 mm to (165.7, 68.6)
- moved C1 118.1 mm to (165.9, 64.9), turned to -90 degrees
- moved R35 118.0 mm to (153.5, 57.5), turned to -90 degrees
- moved C4 113.9 mm to (160.9, 64.9), turned to 90 degrees
- moved C9 113.9 mm to (156.2, 64.9), turned to 90 degrees
- moved C7 112.0 mm to (159.3, 64.9), turned to 90 degrees
- moved R11 107.8 mm to (157.8, 65.4)
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Connections:
- C13 pad 2: +TEMP_VSENSE -> LTEMP_VSENSE
- C17 pad 1: +MOTOR_VBAT -> +LMOTOR_VBAT
- C22 pad 1: +MOTOR_VBAT -> +RMOTOR_VBAT
- D10 pad 1: GND -> +LMOTOR_VBAT
- D10 pad 2: Net-(D10-Pad2) -> Net-(C18-Pad2)
- D11 pad 1: Net-(R17-Pad2) -> Net-(C18-Pad2)
- D11 pad 2: Net-(Q1-Pad3) -> GND
- D18 pad 1: Net-(R24-Pad2) -> +RMOTOR_VBAT
- D18 pad 2: Net-(Q5-Pad3) -> Net-(C23-Pad2)
- D19 pad 1: Net-(R25-Pad1) -> Net-(C23-Pad2)
- D19 pad 2: Net-(Q6-Pad3) -> GND
- Q1 pad 1: +MOTOR_VBAT -> +LMOTOR_VBAT
- Q1 pad 2: +MOTOR_VBAT -> +LMOTOR_VBAT
- Q1 pad 5: +MOTOR_VBAT -> +LMOTOR_VBAT
- Q1 pad 6: +MOTOR_VBAT -> +LMOTOR_VBAT
- Q1 pad 7: +MOTOR_VBAT -> +LMOTOR_VBAT
- Q3 pad 1: +MOTOR_VBAT -> +LMOTOR_VBAT
- Q3 pad 2: +MOTOR_VBAT -> +LMOTOR_VBAT
- Q3 pad 5: +MOTOR_VBAT -> +LMOTOR_VBAT
- Q3 pad 6: +MOTOR_VBAT -> +LMOTOR_VBAT
- Q3 pad 7: +MOTOR_VBAT -> +LMOTOR_VBAT
- Q5 pad 1: +MOTOR_VBAT -> +RMOTOR_VBAT
- Q5 pad 2: +MOTOR_VBAT -> +RMOTOR_VBAT
- Q5 pad 5: +MOTOR_VBAT -> +RMOTOR_VBAT
- Q5 pad 6: +MOTOR_VBAT -> +RMOTOR_VBAT
- Q5 pad 7: +MOTOR_VBAT -> +RMOTOR_VBAT
- Q7 pad 1: +MOTOR_VBAT -> +RMOTOR_VBAT
- Q7 pad 2: +MOTOR_VBAT -> +RMOTOR_VBAT
- Q7 pad 5: +MOTOR_VBAT -> +RMOTOR_VBAT
- Q7 pad 6: +MOTOR_VBAT -> +RMOTOR_VBAT
- Q7 pad 7: +MOTOR_VBAT -> +RMOTOR_VBAT
- R16 pad 1: +MOTOR_VBAT -> +LMOTOR_VBAT
- R23 pad 1: +MOTOR_VBAT -> +RMOTOR_VBAT
- R35 pad 1: Net-(D10-Pad2) -> Net-(D6-Pad2)
- R4 pad 2: +MOTOR_VBAT -> +LMOTOR_VBAT
- R5 pad 2: +MOTOR_VBAT -> +LMOTOR_VBAT
- U2 pad 1: MOTOR_ISENSE -> LMOTOR_ISENSE
- U7 pad 2: +TEMP_VSENSE -> LTEMP_VSENSE
- U8 pad 15: RMOTOR_FORWARD -> LTEMP_VSENSE
- U8 pad 16: RMOTOR_BACKWARDS -> RTEMP_VSENSE
- U8 pad 27: unconnected-(U8-Pad27) -> RMOTOR_FORWARD
- U8 pad 28: LMOTOR_FORWARD -> RMOTOR_BACKWARDS
- U8 pad 30: unconnected-(U8-Pad30) -> LMOTOR_FORWARD
- U8 pad 7: +TEMP_VSENSE -> LTEMP_VSENSE
- U8 pad 9: MOTOR_ISENSE -> RMOTOR_ISENSE
Routing:
- added copper zone on In2.Cu, net GND
Other:
- copper layers 2 -> 4

Commit message: my god
my god
Parts:
- C1, C4, C5, C7, D1, D2, D3, D4, J1, L1, R30, R31, R34, R6, R7, R9, U1: moved to B.Cu
- R11: value 16.5k -> 52.3k; moved to B.Cu
- R12: value 10k -> 16.5k; moved to B.Cu
- U4: value LP38692MP-ADJ -> AP7366-W5-7; footprint Package_TO_SOT_SMD:SOT-223-5 -> Footprints:AP7366-W5-7; moved to B.Cu
- moved R37 123.9 mm to (161.2, 92.3)
- moved C26 121.1 mm to (154.2, 110.0)
- moved R36 121.1 mm to (149.0, 111.9)
- moved R38 121.1 mm to (158.4, 106.2)
- moved U14 121.1 mm to (154.3, 106.8)
- moved C27 121.1 mm to (158.2, 110.0)
- moved D3 82.2 mm to (138.5, 89.2), turned to 90 degrees
- moved U2 81.6 mm to (119.0, 101.8)
- moved U13 81.2 mm to (126.1, 108.1), turned to -90 degrees
- moved C6 77.5 mm to (106.6, 111.7)
- moved C2 77.5 mm to (115.8, 107.0)
- moved C3 77.5 mm to (124.8, 100.6)
- moved C8 77.5 mm to (114.6, 112.2)
- moved R3 77.5 mm to (110.6, 112.2)
- moved R33 77.5 mm to (146.0, 100.6)
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Connections:
- C15 pad 1: +VDD -> +VDD_L
- C16 pad 1: LBOOTSTRAP -> LLBOOTSTRAP
- C18 pad 1: RBOOTSTRAP -> LRBOOTSTRAP
- C19 pad 1: +VDD -> +VDD_L
- C20 pad 1: +VDD -> +VDD_R
- C21 pad 1: LBOOTSTRAP -> RLBOOTSTRAP
- C23 pad 1: RBOOTSTRAP -> RRBOOTSTRAP
- C24 pad 1: +VDD -> +VDD_R
- J4 pad 2: Net-(J4-Pad2) -> /USB/DN
- J4 pad 3: Net-(J4-Pad3) -> /USB/DP
- R14 pad 2: +VDD -> +VDD_L
- R15 pad 2: +VDD -> +VDD_L
- R16 pad 2: +VDD -> +VDD_L
- R21 pad 2: +VDD -> +VDD_R
- R22 pad 2: +VDD -> +VDD_R
- R23 pad 2: +VDD -> +VDD_R
- U10 pad 1: +VDD -> +VDD_L
- U10 pad 2: RBOOTSTRAP -> LRBOOTSTRAP
- U11 pad 1: +VDD -> +VDD_R
- U11 pad 2: LBOOTSTRAP -> RLBOOTSTRAP
- U12 pad 1: +VDD -> +VDD_R
- U12 pad 2: RBOOTSTRAP -> RRBOOTSTRAP
- U4 pad 2: Net-(R11-Pad2) -> GND
- U4 pad 3: +3V3 -> +5V
- U4 pad 4: +5V -> Net-(R11-Pad2)
- U4 pad 5: GND -> +3V3
- U5 pad 1: Net-(J4-Pad3) -> /USB/DP
- U5 pad 2: Net-(J4-Pad3) -> /USB/DN
- U6 pad 1: Net-(J4-Pad3) -> /USB/DP
- U6 pad 12: Net-(J4-Pad2) -> /USB/DN
- U8 pad 15: LTEMP_VSENSE -> LMOTOR_ISENSE
- U8 pad 31: /MCU/LMOTOR_PPM -> /MCU/RMOTOR_PPM
- U8 pad 32: /MCU/RMOTOR_PPM -> /MCU/LMOTOR_PPM
- U9 pad 1: +VDD -> +VDD_L
- U9 pad 2: LBOOTSTRAP -> LLBOOTSTRAP
Routing:
- net Net-(C23-Pad2): track 0.00 -> 32.2 mm, vias 0 -> 2
- net GND: track 0.00 -> 31.3 mm, vias 0 -> 167
- net Net-(C18-Pad2): track 0.00 -> 29.9 mm, vias 0 -> 2
- net Net-(C21-Pad2): track 0.00 -> 29.8 mm, vias 0 -> 2
- net Net-(C16-Pad2): track 0.00 -> 27.5 mm, vias 0 -> 2
- net +RMOTOR_VBAT: track 0.00 -> 21.1 mm, vias 0 -> 84
- net +LMOTOR_VBAT: track 0.00 -> 18.3 mm, vias 0 -> 81
- net +VDD_L: track 0.00 -> 18.1 mm, vias 0 -> 2
- net +VDD_R: track 0.00 -> 17.6 mm, vias 0 -> 2
- net +3V3: track 0.00 -> 12.3 mm
- net +5V: track 0.00 -> 12.3 mm
- net /POWER/+BATT: track 0.00 -> 10.4 mm, vias 0 -> 24
- net Net-(D20-Pad1): track 0.00 -> 8.44 mm, vias 0 -> 2
- net Net-(D14-Pad1): track 0.00 -> 7.60 mm, vias 0 -> 2
- net Net-(D12-Pad1): track 0.00 -> 7.54 mm, vias 0 -> 2
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- added copper zone on B.Cu, net +LMOTOR_VBAT
- added copper zone on In1.Cu, net +LMOTOR_VBAT
- added copper zone on In1.Cu, net +RMOTOR_VBAT
- added copper zone on In3.Cu, net /POWER/+BATT
- added copper zone on B.Cu, net Net-(C16-Pad2)
- added copper zone on B.Cu, net Net-(C18-Pad2)
- added copper zone on B.Cu, net Net-(C21-Pad2)
- added copper zone on B.Cu, net Net-(C23-Pad2)
- added copper zone on B.Cu, net Net-(C4-Pad2)
Other:
- board size 50.8 x 19 mm -> 63.5 x 19 mm
- copper layers 4 -> 6

Commit message: The monstrosity is almost done
The monstrosity is almost done
Parts:
- removed R14, R21: 0, Resistor_SMD:R_0402_1005Metric
- C28, C29, C6, C8, C9, R1, R10, R2, R39, R8, U15, U3, U7: moved to B.Cu
- C7: moved to F.Cu
- moved R10 40.5 mm to (127.2, 81.9), turned to 180 degrees
- moved C6 38.6 mm to (130.3, 81.2), turned to 180 degrees
- moved U7 36.9 mm to (109.2, 85.7), turned to 180 degrees
- moved R32 36.8 mm to (124.0, 73.6)
- moved R2 36.5 mm to (132.0, 85.9), turned to 90 degrees
- moved R33 33.9 mm to (124.0, 74.8)
- moved U3 33.8 mm to (131.0, 83.2)
- moved C8 32.5 mm to (128.8, 82.9), turned to 90 degrees
- moved C25 31.6 mm to (118.3, 85.1), turned to 90 degrees
- moved C12 31.2 mm to (109.9, 85.7)
- moved C13 31.1 mm to (109.0, 86.8)
- moved R13 31.0 mm to (109.0, 84.5)
- moved R1 30.3 mm to (133.1, 85.9), turned to -90 degrees
- moved R8 25.0 mm to (127.2, 83.0)
- moved U13 24.7 mm to (123.5, 83.5), turned to 180 degrees
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Connections:
- R37 pad 1: /POWER/+BATT -> +RMOTOR_VBAT
- R37 pad 2: +RMOTOR_VBAT -> /POWER/+BATT
Routing:
- net GND: track 31.3 -> 46.6 mm, vias 167 -> 171
- net +3V3: track 12.3 -> 18.7 mm, vias 0 -> 1
- net Net-(C3-Pad2): track 0.00 -> 5.18 mm
- net Net-(C27-Pad1): track 0.00 -> 4.46 mm
- net Net-(C27-Pad2): track 0.00 -> 3.78 mm
- net FLASH_MOSI: track 0.00 -> 3.13 mm, vias 0 -> 1
- net /POWER/+BATT: track 10.4 -> 13.3 mm
- net Net-(C28-Pad2): track 0.00 -> 2.53 mm
- net +LMOTOR_VBAT: track 18.3 -> 20.7 mm, vias 81 -> 67
- net Net-(C3-Pad1): track 0.00 -> 2.31 mm
- net +RMOTOR_VBAT: track 21.1 -> 23.3 mm, vias 84 -> 70
- net Net-(D6-Pad2): track 0.00 -> 2.15 mm
- net Net-(C12-Pad2): track 0.00 -> 2.01 mm, vias 0 -> 1
- net +5V: track 12.3 -> 14.2 mm, vias 0 -> 1
- net RTEMP_VSENSE: track 0.00 -> 1.42 mm
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
Commit message: ahhhhh
Parts:
- removed R32, R33: 0, Resistor_SMD:R_0402_1005Metric
- moved U3 5.39 mm to (136.0, 85.3)
- moved C8 4.00 mm to (132.7, 83.4)
Connections:
- U13 pad 3: Net-(R32-Pad1) -> unconnected-(U13-Pad3)
- U13 pad 7: Net-(R33-Pad2) -> unconnected-(U13-Pad7)
- U8 pad 15: LMOTOR_ISENSE -> RMOTOR_ISENSE
- U8 pad 27: RMOTOR_FORWARD -> RMOTOR_BACKWARDS
- U8 pad 28: RMOTOR_BACKWARDS -> RMOTOR_FORWARD
- U8 pad 29: LMOTOR_BACKWARDS -> LMOTOR_FORWARD
- U8 pad 30: LMOTOR_FORWARD -> LMOTOR_BACKWARDS
- U8 pad 9: RMOTOR_ISENSE -> LMOTOR_ISENSE
Routing:
- net +3V3: track 18.7 -> 61.0 mm, vias 1 -> 12
- net LTEMP_VSENSE: track 1.04 -> 38.5 mm
- net LMOTOR_BACKWARDS: track 0.00 -> 34.8 mm, vias 0 -> 3
- net FLASH_SCK: track 0.00 -> 30.5 mm, vias 0 -> 2
- net LMOTOR_FORWARD: track 0.00 -> 29.9 mm, vias 0 -> 3
- net LMOTOR_ISENSE: track 0.00 -> 27.7 mm
- net RMOTOR_FORWARD: track 0.00 -> 27.5 mm, vias 0 -> 4
- net FLASH_MOSI: track 3.13 -> 30.5 mm, vias 1 -> 2
- net RMOTOR_ISENSE: track 0.00 -> 26.7 mm, vias 0 -> 2
- net RMOTOR_BACKWARDS: track 0.00 -> 26.5 mm, vias 0 -> 4
- net +5V: track 14.2 -> 31.7 mm, vias 1 -> 11
- net FLASH_MISO: track 0.00 -> 15.0 mm, vias 0 -> 2
- net RTEMP_VSENSE: track 1.42 -> 13.0 mm, vias 0 -> 1
- net ~{FLASH_CS}: track 0.00 -> 11.4 mm, vias 0 -> 2
- net Net-(C8-Pad1): track 0.00 -> 11.2 mm
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- added copper zone on In1.Cu, net +3V3
- added copper zone on In3.Cu, net +3V3
- added copper zone on B.Cu, net +5V
- added copper zone on In1.Cu, net +5V
- added copper zone on B.Cu, net +XT_VBAT
- added copper zone on B.Cu, net /POWER/+BATT
- added copper zone on B.Cu, net GND
- added copper zone on F.Cu, net GND
