File: MotorController/MotorController.kicad_sch (KiCad schematic)
At the start: 3 parts, among them J1 Conn_01x02, J2 Conn_01x02, J3 Conn_01x03

Commit message: ahhhhh
Other:
- sheet FLASH ports: added none; removed ~{FLASH_HOLD}, ~{FLASH_W}
Changed lines of the file:
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@@
       (effects (font (size 1.27 1.27)) (justify right))
-    )
-    (pin "~{FLASH_W}" input (at 185.42 88.9 180)
-      (effects (font (size 1.27 1.27)) (justify left))
-    )
-    (pin "~{FLASH_HOLD}" input (at 185.42 86.36 180)
-      (effects (font (size 1.27 1.27)) (justify left))
     )
   )
@@
       (reference "R31") (unit 1) (value "19.1") (footprint "Resistor_SMD:R_0402_1005Metric")
     )
-    (path "/33d17ea3-a408-483c-9d51-34e840ff36fb/56f58402-6224-4f2e-a240-16b1052d8916"
-      (reference "R32") (unit 1) (value "0") (footprint "Resistor_SMD:R_0402_1005Metric")
-    )
-    (path "/33d17ea3-a408-483c-9d51-34e840ff36fb/2ce3b724-983d-4634-a0e4-3ca6ba3131eb"
-      (reference "R33") (unit 1) (value "0") (footprint "Resistor_SMD:R_0402_1005Metric")
-    )
     (path "/cd9205e1-9dd8-4849-8d2c-a52a0d3ed8fe/054cda4b-a8ba-41b1-8ca3-c2e99d0199d8"
